File: 03_Development/Hardware/Proto_Bluetooth/Board_Bluetooth_radio_platform.kicad_pcb (KiCad board)
At the start: 2 copper layers, 232.5 x 124.5 mm, 99 parts, among them J1 Conn_01x02, J10 Conn_01x03, J11 HMI_rotaryEncoder_1, J12 HMI_rotaryEncoder_1, J13 Conn_01x08_epaper, J14 Conn_01x03_fmModule_audioOutp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, J15 Conn_01x02_classD_SD, J16 Conn_02x12_Odd_Even, J19 Conn_01x02_rn52_usb, J2 Conn_01x08, J20 Conn_01x05_toClassD, J3 BT_RN52_connector_left, J4 Conn_01x02, J5 BT_RN52_connector_right, J6 FM_interface, J7 BT_debug_connector, J8 BT_extension_connector, J9 SYS_debug_connector, SW1 SW_Push, U1 LM317_TO-220, U3 TPA6112A2DGQ, U4 TS5A2234

Commit message: [HDW_29] Fixed LM317 heatsink PCB space
LM317 has a heeatsink in case of too much power disspation.
Its sie is approximately 20x20 mm and has influence on
mechanical place of other components.
Moved power supply unit so that all is good
Parts:
- U1: footprint Package_TO_SOT_THT:TO-220-3_Vertical -> Package_TO_SOT_THT:TO-220-3_Horizontal_TabDown
- moved C1 31.5 mm to (142.5, 48.4), turned to 90 degrees
- moved J_sys1 26.1 mm to (132.6, 44.4)
- moved C4 20.0 mm to (124.3, 53.8)
- moved R11 20.0 mm to (124.5, 46.5)
- moved R14 20.0 mm to (126.8, 53.8)
- moved C5 20.0 mm to (108.4, 53.7)
- moved C6 20.0 mm to (131.8, 53.8)
- moved C7 20.0 mm to (115.9, 53.7)
- moved J11 20.0 mm to (130.6, 49.3)
- moved JRP2040R_1 20.0 mm to (131.4, 60.8)
- moved JRP4020L_1 20.0 mm to (83.2, 78.6)
- moved R12 20.0 mm to (108.7, 46.5)
- moved R13 20.0 mm to (129.3, 53.8)
- moved R15 20.0 mm to (113.4, 53.7)
- moved R16 20.0 mm to (110.9, 53.7)
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Routing:
- net Net-(C1-Pad1): track 11.3 -> 38.7 mm
- net FM_SEN: track 10.2 -> 31.3 mm
- net sys_button_b: track 119.7 -> 100.0 mm
- net sys_button_a: track 143.7 -> 124.0 mm
- net sys_onoff_o: track 16.8 -> 36.0 mm
- net SYS_audio_sw: track 121.5 -> 102.8 mm
- net FM_GPIO1: track 25.7 -> 7.61 mm
- net FM_SDIO: track 8.63 -> 21.1 mm
- net sys_Vsys: track 72.8 -> 60.5 mm
- net BT_GPIO2: track 119.2 -> 107.7 mm
- net FM_RST: track 26.2 -> 37.5 mm
- net FM_SCLK: track 9.85 -> 19.9 mm
- net Net-(J15-Pad1): track 5.37 -> 15.4 mm
- net EPD_DC: track 38.6 -> 48.5 mm
- net EPD_DIN: track 19.7 -> 29.4 mm
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
Commit message: [HDW_31] Fixed add of trim resistance
Power supply with LM317 is not always perfect with
10% resistances. Add of potentiometer to get better
3.3 V values
Parts:
- removed R5: 390, Resistor_SMD:R_0805_2012Metric_Pad1.20x1.40mm_HandSolder
- removed R6: 330, Resistor_SMD:R_0805_2012Metric_Pad1.20x1.40mm_HandSolder
- added RV1: R_Potentiometer_Trim, Potentiometer_THT:Potentiometer_Bourns_3299W_Vertical, F.Cu at (173.0, 50.9)
- moved F1 4.13 mm to (179.1, 38.3)
- moved C3 3.19 mm to (166.6, 50.8)
- moved R8 3.08 mm to (166.6, 46.0)
- moved D1 1.78 mm to (184.7, 42.2)
Routing:
- net +3V3: track 596.2 -> 582.4 mm
- net Net-(R8-Pad2): track 20.0 -> 26.1 mm
- net Net-(R5-Pad2): track 3.06 -> 0.00 mm
- net Net-(D1-Pad1): track 5.33 -> 7.13 mm
- net sys_onoff_o: track 36.0 -> 34.2 mm

Commit message: [HDW_31] Add 1205V DC DC converter
Add of a murata NXE2S1205MC DC DC downconverter
to add 12V power supply possibility. Will maybe
not be soldered but footprints are there for
future amelioration. Helps to plug a battery
on radio
Parts:
- added J17: Conn_01x02, Connector_PinSocket_2.54mm:PinSocket_1x02_P2.54mm_Vertical, F.Cu at (152.1, 125.0)
- added L1: L_Coupled_1243 22n, Inductor_SMD:L_Wuerth_WE-DD-Typ-M-Typ-S, F.Cu at (142.0, 111.0)
- added U2: NXE2S1205MC, Converter_DCDC:Converter_DCDC_Murata_NXExSxxxxMC_SMD, F.Cu at (141.9, 122.6)
- moved D1 2.03 mm to (184.7, 40.1)
Routing:
- net sys_onoff_i: track 12.0 -> 129.9 mm
- net Net-(U2-Pad7): track 0.00 -> 14.2 mm
- net Net-(U2-Pad8): track 0.00 -> 13.3 mm
- net Net-(J17-Pad1): track 0.00 -> 5.64 mm
- net Net-(J17-Pad2): track 0.00 -> 5.64 mm
- net +3V3: track 582.4 -> 585.8 mm
- net Net-(D1-Pad1): track 7.13 -> 6.29 mm
- net sys_onoff_o: track 34.2 -> 33.4 mm

Commit message: [HDW_36] Fixed edge cut layer
Edge.cut layer fixed with circle removed
Cleanup TICKET.md file
minor other correction
READY TO TEST. All firmware should be tested
on breadboard first before sending to production
Parts:
- added HS1: Heatsink, Heatsink:Heatsink_AAVID_TV5G_TO220_Horizontal, F.Cu at (152.1, 64.8)
- moved F1 6.38 mm to (178.6, 44.7), turned to 180 degrees
- moved R10 4.44 mm to (166.6, 56.6)
- moved R30 2.62 mm to (155.4, 37.1), turned to 0 degrees
- moved R32 2.61 mm to (134.9, 37.1), turned to 0 degrees
- moved R34 2.60 mm to (114.3, 37.1), turned to 0 degrees
- moved R36 2.59 mm to (93.7, 37.1), turned to 0 degrees
- moved R38 2.58 mm to (73.3, 37.1), turned to 0 degrees
- moved R40 2.56 mm to (52.3, 37.1), turned to 0 degrees
- moved R42 2.53 mm to (32.0, 37.1), turned to 0 degrees
- moved J_pwrLed1 2.12 mm to (170.4, 58.2), turned to 180 degrees
- moved J1 1.95 mm to (213.9, 46.2), turned to 90 degrees
- moved R35 1.05 mm to (93.7, 39.6), turned to 180 degrees
- moved R29 0.87 mm to (155.4, 39.6), turned to 180 degrees
- moved R31 0.85 mm to (134.9, 39.6), turned to 180 degrees
- moved R33 0.82 mm to (114.3, 39.6), turned to 180 degrees
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Routing:
- net +3V3: track 585.8 -> 594.4 mm
- net Net-(U2-Pad7): track 14.2 -> 9.15 mm
- net Net-(C1-Pad1): track 38.6 -> 34.7 mm
- net Net-(U2-Pad8): track 13.3 -> 9.41 mm
- net sys_onoff_i: track 129.9 -> 126.8 mm
- net Net-(D1-Pad1): track 6.29 -> 8.88 mm
- net Net-(J_IX1-Pad5): track 5.43 -> 3.66 mm
- net EPD_BUSY: track 19.7 -> 21.2 mm
- net Net-(J_IV1-Pad5): track 5.09 -> 3.59 mm
- net Net-(J_X1-Pad5): track 5.43 -> 3.98 mm
- net Net-(J_V1-Pad5): track 5.09 -> 3.65 mm
- net Net-(J_VI1-Pad5): track 5.08 -> 3.73 mm
- net Net-(J_VII1-Pad5): track 5.05 -> 3.79 mm
- net Net-(J16-Pad5): track 5.08 -> 4.02 mm
- net Net-(J_IV1-Pad1): track 5.41 -> 4.87 mm
Other:
- board size 232.5 x 124.5 mm -> 218 x 124.5 mm
- board text added: "DjenaDev Bt radio V 1.0 08 2023"

Commit message: [HDW_25] Fix mounting holes issue
Add mounting holes for screwing to radio chassis
Add mounting holes for PAM8302
Cleanup TICKETS file
Change README name
Parts:
- removed HS1: Heatsink, Heatsink:Heatsink_AAVID_TV5G_TO220_Horizontal
- added REF1: MountingHole_2.2mm_M2_DIN965, MountingHole:MountingHole_2.2mm_M2_DIN965, F.Cu at (39.5, 25.5)
- added REF2: MountingHole_2.2mm_M2_DIN965, MountingHole:MountingHole_2.2mm_M2_DIN965, F.Cu at (100.5, 25.5)
- added REF3: MountingHole_2.2mm_M2_DIN965, MountingHole:MountingHole_2.2mm_M2_DIN965, F.Cu at (202.5, 25.5)
- added REF4: MountingHole_2.5mm, MountingHole:MountingHole_2.5mm, F.Cu at (83.1, 102.7)
- added REF5: MountingHole_2.5mm, MountingHole:MountingHole_2.5mm, F.Cu at (93.6, 102.7)
Routing:
- net BT_MIC_L-: track 39.9 -> 37.1 mm
- net sys_button_a: track 124.0 -> 121.3 mm
- net sys_button_b: track 100.0 -> 97.3 mm
- net GND: track 4.80 -> 2.73 mm
- net BT_SPKR_R-: track 31.7 -> 29.7 mm
- net BT_SPKR_R+: track 25.9 -> 24.3 mm
- net BT_PWREN: track 53.6 -> 52.6 mm
- net /audio_amp_stage/SPKR-: track 24.8 -> 24.1 mm
- net /audio_amp_stage/SPKR+: track 19.6 -> 19.1 mm
- net Net-(J12-Pad1): track 4.26 -> 3.76 mm
Other:
- board size 218 x 124.5 mm -> 218 x 124 mm
