File: 03_Development/Hardware/Proto_Bluetooth/Board_Bluetooth_radio_platform.kicad_pcb (KiCad board)
At the start: 2 copper layers, 218 x 124 mm, 106 parts, among them J1 Conn_01x02, J10 Conn_01x03, J11 HMI_rotaryEncoder_1, J12 HMI_rotaryEncoder_1, J13 Conn_01x08_epaper, J14 Conn_01x03_fmModule_audioOutp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, J15 Conn_01x02_classD_SD, J16 Conn_02x12_Odd_Even, J17 Conn_01x02, J19 Conn_01x02_rn52_usb, J2 Conn_01x08, J20 Conn_01x05_toClassD, J3 BT_RN52_connector_left, J4 Conn_01x02, J5 BT_RN52_connector_right, J6 FM_interface, J7 BT_debug_connector, J8 BT_extension_connector, J9 SYS_debug_connector, SW1 SW_Push, U1 LM317_TO-220, U2 NXE2S1205MC, U3 TPA6112A2DGQ, U4 TS5A2234

Commit message: [HDW_38] Fix Bt communication wires
Bluetooth Rx pin connected to GPIO4 of RP240
Bluetooth Tx pin connected to GPIO5 of RP2040
Parts:
- C4, C5, C6, C7: value 10n -> 47n
- R1, R2, R3, R4: value 100K -> 100k
- renumbered J16 to J_VIII1
Connections:
- JRP4020L_1 pad 4: BT_UART_RX -> FM_RST
- JRP4020L_1 pad 5: BT_UART_TX -> FM_SEN
- JRP4020L_1 pad 6: FM_RST -> BT_UART_RX
- JRP4020L_1 pad 7: FM_SEN -> BT_UART_TX
Routing:
- net FM_RST: track 37.5 -> 44.6 mm
- net FM_SEN: track 31.1 -> 37.4 mm
- net BT_UART_TX: track 73.1 -> 69.8 mm
- net BT_UART_RX: track 78.3 -> 75.7 mm

Commit message: [HDW_41] FIX communication lines to central unit
FM, EP and BT modules had been routed to ports of RP2040 which don't allow
UART or I2C and must have been changed
Parts:
- C4, C5, C6, C7: value 47n -> 10n
- R1, R11, R12, R2, R28, R29, R3, R30, R31, R32, R33, R34, R35, R36, R37, R38, R39, R4, R40, R41, R42: value 100k -> 10k
- R13, R14, R15, R16: value 470k -> 10k
- moved J13 3.00 mm to (141.2, 98.3)
Connections:
- JRP4020L_1 pad 10: FM_SCLK -> FM_GPIO1
- JRP4020L_1 pad 11: EPD_DC -> BT_UART_RX
- JRP4020L_1 pad 12: EPD_CS -> BT_UART_TX
- JRP4020L_1 pad 19: FM_GPIO2 -> EPD_DC
- JRP4020L_1 pad 20: FM_GPIO1 -> EPD_CS
- JRP4020L_1 pad 6: BT_UART_RX -> FM_SDIO
- JRP4020L_1 pad 7: BT_UART_TX -> FM_SCLK
- JRP4020L_1 pad 9: FM_SDIO -> FM_GPIO2
Routing:
- net FM_SDIO: track 20.9 -> 71.2 mm
- net FM_SCLK: track 19.9 -> 64.6 mm
- net FM_GPIO1: track 7.61 -> 40.7 mm
- net FM_GPIO2: track 15.4 -> 44.4 mm
- net EPD_CS: track 43.6 -> 34.6 mm
- net BT_UART_TX: track 69.8 -> 78.7 mm
- net EPD_DC: track 48.5 -> 39.6 mm
- net BT_UART_RX: track 75.7 -> 81.7 mm
- net EPD_CLK: track 33.9 -> 30.9 mm
- net EPD_RST: track 24.8 -> 21.8 mm
- net EPD_DIN: track 29.4 -> 26.4 mm
- net EPD_BUSY: track 21.2 -> 18.4 mm
- net FM_RST: track 44.6 -> 41.8 mm, vias 0 -> 1

Commit message: [HDW_45] FIX remove of 12V power supply
Parts:
- removed J17: Conn_01x02, Connector_PinSocket_2.54mm:PinSocket_1x02_P2.54mm_Vertical
- removed L1: L_Coupled_1243 22n, Inductor_SMD:L_Wuerth_WE-DD-Typ-M-Typ-S
- removed U2: NXE2S1205MC, Converter_DCDC:Converter_DCDC_Murata_NXExSxxxxMC_SMD
Routing:
- net sys_onoff_i: track 126.8 -> 12.2 mm
- net Net-(L1-Pad1): track 9.41 -> 0.00 mm
- net Net-(L1-Pad4): track 9.15 -> 0.00 mm
- net Net-(J17-Pad1): track 5.64 -> 0.00 mm
- net Net-(J17-Pad2): track 5.64 -> 0.00 mm

Commit message: [HDW_43] FIX PCB edges for mechanical fit in Radio
Left side is not fully filled as we need a space for Bluetooth
antenna's
Space for loudspeaker had to be increased
Right upper size had to be reduced of a couple of cm
Left spaces had some space avaialble which is now used
Ready for button resync and replace of components
Parts:
- moved C2 59.9 mm to (221.2, 47.3)
- moved C3 59.9 mm to (226.5, 49.7)
- moved D1 59.9 mm to (244.6, 39.1)
- moved J1 59.9 mm to (273.8, 45.1)
- moved J11 59.9 mm to (190.5, 48.3)
- moved J15 59.9 mm to (136.3, 93.2)
- moved J3 59.9 mm to (132.6, 101.5)
- moved J_I1 59.9 mm to (272.7, 33.4)
- moved J_III1 59.9 mm to (231.4, 33.4)
- moved J_VIII1 59.9 mm to (128.2, 33.4)
- moved J_pwrLed1 59.9 mm to (230.3, 57.1)
- moved R10 59.9 mm to (226.5, 55.6)
- moved R28 59.9 mm to (171.0, 64.2)
- moved R31 59.9 mm to (194.8, 38.6)
- moved R32 59.9 mm to (194.8, 36.0)
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Other:
- board size 218 x 124 mm -> 220.5 x 124 mm

Commit message: [HDW_44][HDW_42][HDW_50] FIX all of those topics
Move mounting hole to their correct place
Push buttons are good and works as expected
Place of specific headers for push-buttons is now corrected
Parts:
- moved C1 98.1 mm to (266.7, 121.4), turned to -90 degrees
- moved D1 92.8 mm to (224.5, 129.7), turned to 90 degrees
- moved U1 84.8 mm to (254.7, 121.6), turned to 0 degrees
- moved F1 81.8 mm to (230.6, 125.1), turned to 0 degrees
- moved R8 80.5 mm to (242.5, 123.8), turned to -90 degrees
- moved C2 78.8 mm to (247.9, 121.4), turned to -90 degrees
- moved R2 73.2 mm to (91.5, 101.7)
- moved J19 73.2 mm to (98.3, 98.5)
- moved JGPIO7 73.2 mm to (108.0, 98.5)
- moved JGPIO9 73.2 mm to (91.6, 98.5)
- moved R1 73.2 mm to (86.6, 101.7)
- moved R3 73.2 mm to (103.0, 101.7)
- moved R4 73.2 mm to (108.0, 101.7)
- moved C3 71.1 mm to (242.5, 119.0), turned to 90 degrees
- moved RV1 69.1 mm to (236.2, 118.9), turned to 0 degrees
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Routing:
- net +3V3: track 594.1 -> 490.2 mm
- net BT_GPIO6: track 133.4 -> 40.2 mm, vias 1 -> 0
- net Net-(J19-Pad2): track 69.1 -> 1.64 mm
- net Net-(J19-Pad1): track 68.1 -> 2.62 mm
- net BT_GPIO2: track 107.7 -> 45.5 mm
- net BT_GPIO9: track 64.2 -> 3.28 mm
- net BT_GPIO7: track 62.0 -> 1.67 mm
- net sys_button_a: track 121.3 -> 85.9 mm
- net BT_MIC_L+: track 34.9 -> 0.00 mm
- net sys_button_b: track 97.3 -> 63.0 mm
- net BT_MIC_R-: track 42.8 -> 13.3 mm
- net BT_LED_0: track 32.1 -> 2.94 mm
- net DBG_UART_RX: track 31.0 -> 5.05 mm
- net sys_onoff_o: track 33.4 -> 7.50 mm
- net BT_PWREN: track 52.6 -> 27.5 mm
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
Commit message: [HDW_49] FIX place of elements for new version
Remove micro i/o from RN52 as they won't be used
Move power supply down on PCB
Move class D amplifier
Add hole for push buttons mounting
Parts:
- J8: value BT_extension_connector -> Conn_02x06_Counter_Clockwise; footprint Connector_PinSocket_2.54mm:PinSocket_2x08_P2.54mm_Vertical -> Connector_PinSocket_2.54mm:PinSocket_2x06_P2.54mm_Vertical
- moved C1 127.6 mm to (140.1, 105.7), turned to 90 degrees
- moved U1 104.0 mm to (152.0, 105.5), turned to 180 degrees
- moved C2 90.4 mm to (158.9, 105.7), turned to 90 degrees
- moved R8 81.0 mm to (164.2, 103.3), turned to 90 degrees
- moved C3 79.1 mm to (164.2, 108.1), turned to -90 degrees
- moved R10 78.3 mm to (164.2, 114.0), turned to 90 degrees
- moved J9 74.6 mm to (196.8, 60.0)
- moved J_pwrLed1 70.8 mm to (168.0, 115.5), turned to 180 degrees
- moved J10 69.3 mm to (189.5, 65.0), turned to 180 degrees
- moved RV1 66.5 mm to (170.5, 108.2), turned to 180 degrees
- moved F1 59.1 mm to (176.1, 102.0), turned to 180 degrees
- moved D1 53.1 mm to (182.2, 97.5), turned to -90 degrees
- moved R7 50.4 mm to (71.4, 47.8), turned to 180 degrees
- moved D2 45.9 mm to (70.6, 53.9), turned to 90 degrees
- moved R9 44.4 mm to (77.5, 47.8), turned to 0 degrees
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Connections:
- J5 pad 5: BT_MIC_R- -> unconnected-(J5-Pad5)
- J5 pad 6: BT_MIC_L- -> unconnected-(J5-Pad6)
- J5 pad 7: BT_MIC_R+ -> unconnected-(J5-Pad7)
- J5 pad 8: BT_MIC_L+ -> unconnected-(J5-Pad8)
- J5 pad 9: BT_MIC_BIAS -> unconnected-(J5-Pad9)
- J8 pad 1: BT_MIC_R- -> GND
- J8 pad 10: BT_SPI_MOSI -> BT_SPI_SCK
- J8 pad 11: BT_PCM_OUT -> BT_PCM_SYNC
- J8 pad 12: BT_SPI_SCK -> BT_SPI_MISO
- J8 pad 2: BT_MIC_L- -> +3V3
- J8 pad 3: BT_MIC_R+ -> BT_GPIO6
- J8 pad 4: BT_MIC_L+ -> BT_SPI_SS
- J8 pad 5: BT_MIC_BIAS -> GND
- J8 pad 6: BT_GPIO6 -> BT_PCM_CLK
- J8 pad 7: +3V3 -> BT_PCM_IN
- J8 pad 8: GND -> BT_SPI_MOSI
- J8 pad 9: BT_PCM_IN -> BT_PCM_OUT
Routing:
- net sys_onoff_o: track 7.50 -> 147.9 mm
- net +3V3: track 490.2 -> 625.6 mm
- net BT_GPIO6: track 40.2 -> 127.0 mm
- net BT_GPIO2: track 45.5 -> 113.0 mm, vias 0 -> 1
- net DBG_UART_RX: track 5.05 -> 66.5 mm
- net DBG_UART_TX: track 17.1 -> 64.9 mm
- net BT_PWREN: track 27.5 -> 68.2 mm
- net BT_PCM_IN: track 42.4 -> 12.0 mm
- net SYS_audio_sw: track 79.2 -> 108.3 mm
- net BT_PCM_OUT: track 37.2 -> 8.42 mm
- net BT_PCM_SYNC: track 32.2 -> 5.35 mm
- net sys_button_a: track 85.9 -> 106.8 mm
- net sys_button_b: track 63.0 -> 82.9 mm
- net sys_onoff_i: track 0.00 -> 19.5 mm
- net BT_MIC_BIAS: track 17.6 -> 0.00 mm
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Other:
- board text added: "DjenaDev Bt radio V 1.1 08 2023"
- board text removed: "DjenaDev Bt radio V 1.0 08 2023"

Commit message: [HDW_51] FIX push button connector
Push button connector for power supply was not a holding
one and had to be changed to a holding one
PCB updated
Add of GND to some of the headers
Parts:
- added REF6: MountingHole_2.2mm_M2_DIN965, MountingHole:MountingHole_2.2mm_M2_DIN965, F.Cu at (218.5, 25.9)
- moved J1 55.9 mm to (208.5, 50.8), turned to 0 degrees
Connections:
- J_I1 pad 2: unconnected-(J_I1-Pad2) -> GND
- J_I1 pad 3: sys_onoff_i -> sys_contact_ai
- J_I1 pad 5: sys_onoff_o -> sys_contact_ao
- J_II1 pad 2: unconnected-(J_II1-Pad2) -> GND
- J_II1 pad 3: sys_contact_bi -> sys_onoff_i
- J_II1 pad 5: sys_contact_bo -> sys_onoff_o
- J_III1 pad 2: unconnected-(J_III1-Pad2) -> GND
Routing:
- net sys_onoff_i: track 19.5 -> 56.9 mm
- net sys_onoff_o: track 147.9 -> 120.4 mm
- net SYS_audio_sw: track 108.3 -> 105.5 mm
- net BT_SPKR_R-: track 29.7 -> 27.8 mm
