File: 03_Development/Hardware/Proto_Bluetooth/Board_Bluetooth_radio_platform.kicad_pcb (KiCad board)
At the start: 2 copper layers, 220.5 x 124 mm, 104 parts, among them J1 Conn_01x02, J10 Conn_01x03, J11 HMI_rotaryEncoder_1, J12 HMI_rotaryEncoder_1, J13 Conn_01x08_epaper, J14 Conn_01x03_fmModule_audioOutp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, J15 Conn_01x02_classD_SD, J19 Conn_01x02_rn52_usb, J2 Conn_01x08, J20 Conn_01x05_toClassD, J3 BT_RN52_connector_left, J4 Conn_01x02, J5 BT_RN52_connector_right, J6 FM_interface, J7 BT_debug_connector, J8 Conn_02x06_Counter_Clockwise, J9 SYS_debug_connector, SW1 SW_Push, U1 LM317_TO-220, U3 TPA6112A2DGQ, U4 TS5A2234

Commit message: RELEASE CANDIDATE V1.1 of PCB
All changes required on schematic and PCB are done
DRC executed
Minimal finalization of PCB with small correction
Ready to be tested before prod
Parts:
- moved C4 1.50 mm to (177.7, 52.7)
- moved C6 1.50 mm to (185.2, 52.7)
- moved J11 1.50 mm to (184.0, 48.3)
- moved R11 1.50 mm to (178.0, 45.4)
- moved R13 1.50 mm to (182.7, 52.7)
- moved R14 1.50 mm to (180.2, 52.7)
Routing:
- net sys_button_a: track 106.8 -> 86.9 mm
- net sys_button_b: track 82.9 -> 64.7 mm
- net +3V3: track 625.5 -> 619.6 mm
- net BT_SPKR_L+: track 21.2 -> 25.2 mm
- net DBG_UART_RX: track 66.5 -> 69.4 mm
- net DBG_RST: track 43.9 -> 42.3 mm
- net RE1_SW: track 18.1 -> 16.6 mm
- net BT_SPI_MISO: track 8.75 -> 7.55 mm
- net BT_SPI_SCK: track 11.4 -> 10.2 mm
- net RE1_A: track 13.6 -> 14.6 mm
- net BT_SPI_MOSI: track 13.8 -> 14.7 mm
- net RE1_B: track 9.80 -> 10.4 mm
- net BT_PCM_SYNC: track 5.35 -> 4.83 mm
- net FM_GPIO2: track 44.4 -> 43.9 mm
- net BT_SPKR_R+: track 24.3 -> 23.8 mm, vias 1 -> 0
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
Commit message: [HDW_54] FIX Bill Of Matierial for V1.1
FIX footprint of C15 and C16 from 0805 to 1210
Order all necessary parts from BOM
Parts:
- C16, C17: footprint Resistor_SMD:R_0805_2012Metric_Pad1.20x1.40mm_HandSolder -> Resistor_SMD:R_1206_3216Metric_Pad1.30x1.75mm_HandSolder
Routing:
- net aud_bt_o-: track 12.4 -> 13.1 mm
- net aud_bt_o+: track 12.2 -> 12.8 mm

Commit message: [HDW_53] FIX layout of audio preamplifier
Parts:
- moved C16 1.69 mm to (96.5, 67.5), turned to 0 degrees
- moved C17 1.49 mm to (96.5, 80.0), turned to 0 degrees
- moved C20 0.75 mm to (102.0, 75.1)
Routing:
- net +3V3: track 619.9 -> 624.3 mm
- net Net-(C16-Pad1): track 6.67 -> 3.66 mm
- net BT_SPKR_R+: track 23.8 -> 26.8 mm
- net BT_PCM_SYNC: track 4.83 -> 7.28 mm
- net aud_bt_o+: track 12.8 -> 10.5 mm
- net aud_bt_o-: track 13.1 -> 11.2 mm
- net GND: track 2.73 -> 4.44 mm, vias 29 -> 30
- net SYS_audio_sw: track 105.5 -> 103.8 mm
- net BT_LED_1: track 10.2 -> 9.29 mm
- net BT_SPKR_R-: track 27.3 -> 28.0 mm

Commit message: [HDW_55] FIX grounding of PCB for better gnd pane
Parts:
- REF1, REF2, REF3, REF6: value MountingHole_2.2mm_M2_DIN965 -> MountingHole; footprint MountingHole:MountingHole_2.2mm_M2_DIN965 -> MountingHole:MountingHole_3.2mm_M3_DIN965
- REF4, REF5: value MountingHole_2.5mm -> MountingHole
Connections:
- J_IV1 pad 2: unconnected-(J_IV1-Pad2) -> GND
- J_IX1 pad 17: unconnected-(J_IX1-Pad17) -> GND
- J_IX1 pad 18: unconnected-(J_IX1-Pad18) -> GND
- J_IX1 pad 8: unconnected-(J_IX1-Pad8) -> GND
- J_V1 pad 2: unconnected-(J_V1-Pad2) -> GND
- J_VIII1 pad 23: unconnected-(J_VIII1-Pad23) -> GND
- J_VIII1 pad 24: unconnected-(J_VIII1-Pad24) -> GND
- J_VIII1 pad 8: unconnected-(J_VIII1-Pad8) -> GND
- J_X1 pad 17: unconnected-(J_X1-Pad17) -> GND
- J_X1 pad 18: unconnected-(J_X1-Pad18) -> GND
- J_X1 pad 8: unconnected-(J_X1-Pad8) -> GND
Routing:
- net Net-(C16-Pad1): track 3.66 -> 6.06 mm
- net Net-(C17-Pad1): track 7.83 -> 7.29 mm
- net GND: vias 30 -> 27

Commit message: PROD Mark II - files sent to production
Modify mechanical placement of buttons and layout
Reduction of pull up/down resistances
Fix communication routing between modules and RP2040
Fix board size
Version: V1.1
Parts:
- moved J1 52.3 mm to (259.8, 40.0), turned to 90 degrees
- moved R29 1.55 mm to (215.0, 38.6)
- moved R30 1.55 mm to (215.0, 36.0)
- moved J_IV1 1.20 mm to (210.6, 33.4)
- moved R31 1.20 mm to (195.0, 38.6)
- moved R32 1.20 mm to (195.0, 36.0)
- moved J_III1 1.10 mm to (231.2, 33.4)
- moved R33 1.10 mm to (174.7, 38.6)
- moved R34 1.10 mm to (174.7, 36.0)
- moved J_V1 1.08 mm to (190.3, 33.4)
- moved C5 1.00 mm to (159.3, 52.6)
- moved C7 1.00 mm to (166.8, 52.6)
- moved J12 1.00 mm to (165.6, 48.3)
- moved J_II1 1.00 mm to (251.7, 33.4)
- moved R12 1.00 mm to (159.6, 45.4)
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Routing:
- net sys_onoff_i: track 56.9 -> 9.67 mm
- net +3V3: track 624.3 -> 612.8 mm
- net sys_onoff_o: track 120.4 -> 128.7 mm
- net sys_Vsys: track 74.5 -> 78.5 mm
- net FM_RST: track 41.1 -> 42.1 mm
- net RE2_SW: track 32.2 -> 33.1 mm
- net RE2_B: track 11.5 -> 12.2 mm
- net sys_button_b: track 64.7 -> 65.3 mm
- net RE2_A: track 11.7 -> 12.2 mm
- net sys_button_a: track 86.9 -> 87.4 mm
- net GND: vias 27 -> 28
Other:
- board size 220.5 x 124 mm -> 220.5 x 121 mm
- board text added: "DjenaDev Bt radio V 1.1 10 2023"
- board text removed: "DjenaDev Bt radio V 1.1 08 2023"
