File: 03_Development/Hardware/Proto_Bluetooth/Board_Bluetooth_radio_platform.kicad_sch (KiCad schematic)
At the start: 48 parts, among them J1 Conn_01x02, J10 Conn_01x03, J11 HMI_rotaryEncoder_1, J12 HMI_rotaryEncoder_1, J19 Conn_01x02_rn52_usb, J2 Conn_01x08, J3 BT_RN52_connector_left, J4 Conn_01x02, J5 BT_RN52_connector_right, J6 FM_interface, J7 BT_debug_connector, J8 BT_extension_connector, J9 SYS_debug_connector, SW1 SW_Push, U1 LM317_TO-220

Commit message: [HDW_29] Fixed LM317 heatsink PCB space
LM317 has a heeatsink in case of too much power disspation.
Its sie is approximately 20x20 mm and has influence on
mechanical place of other components.
Moved power supply unit so that all is good
Parts:
- U1: footprint Package_TO_SOT_THT:TO-220-3_Vertical -> Package_TO_SOT_THT:TO-220-3_Horizontal_TabDown
Changed lines of the file:
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@@
       (effects (font (size 1.27 1.27)) hide)
     )
-    (property "Footprint" "Package_TO_SOT_THT:TO-220-3_Vertical" (id 2) (at 60.96 16.51 0)
+    (property "Footprint" "Package_TO_SOT_THT:TO-220-3_Horizontal_TabDown" (id 2) (at 60.96 16.51 0)
       (effects (font (size 1.27 1.27) italic) hide)
     )
@@
     )
     (path "/350b95f4-a11f-4b8e-a1a2-6edb49986a2d"
-      (reference "U1") (unit 1) (value "LM317_TO-220") (footprint "Package_TO_SOT_THT:TO-220-3_Vertical")
+      (reference "U1") (unit 1) (value "LM317_TO-220") (footprint "Package_TO_SOT_THT:TO-220-3_Horizontal_TabDown")
     )
     (path "/93984d3e-1049-40c4-85f7-3f9031f77d6e/2c8a87db-3d29-497c-8252-401310edddce"

Commit message: [HDW_31] Fixed add of trim resistance
Power supply with LM317 is not always perfect with
10% resistances. Add of potentiometer to get better
3.3 V values
Parts:
- removed R5: 390, Resistor_SMD:R_0805_2012Metric_Pad1.20x1.40mm_HandSolder, symbol Device:R
- removed R6: 330, Resistor_SMD:R_0805_2012Metric_Pad1.20x1.40mm_HandSolder, symbol Device:R
- added RV?: R_Potentiometer_Trim, Potentiometer_THT:Potentiometer_Bourns_3299W_Vertical, symbol Device:R_Potentiometer_Trim
Connections:
- net GND: now also RV?.2, RV?.3
- net at R8.2, U1.1 (ADJ): now also RV?.1
Changed lines of the file:
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@@
     (stroke (width 0) (type default) (color 0 0 0 0))
   )
-  (wire (pts (xy 60.96 51.435) (xy 60.96 53.975))
+  (wire (pts (xy 67.31 40.64) (xy 67.31 46.99))
     (stroke (width 0) (type default) (color 0 0 0 0))
   )
@@
     (stroke (width 0) (type default) (color 0 0 0 0))
   )
-  (wire (pts (xy 60.96 32.385) (xy 60.96 34.29))
+  (wire (pts (xy 60.96 32.385) (xy 60.96 36.83))
     (stroke (width 0) (type default) (color 0 0 0 0))
   )
@@
     (stroke (width 0) (type default) (color 0 0 0 0))
   )
+  (wire (pts (xy 64.77 40.64) (xy 67.31 40.64))
+    (stroke (width 0) (type default) (color 0 0 0 0))
+  )
   (wire (pts (xy 245.11 70.485) (xy 248.92 70.485))
     (stroke (width 0) (type default) (color 0 0 0 0))
@@
     (stroke (width 0) (type default) (color 0 0 0 0))
   )
-  (wire (pts (xy 60.96 41.91) (xy 60.96 43.815))
-    (stroke (width 0) (type default) (color 0 0 0 0))
-  )
   (wire (pts (xy 69.85 106.045) (xy 69.85 107.315))
     (stroke (width 0) (type default) (color 0 0 0 0))
@@
     (stroke (width 0) (type default) (color 0 0 0 0))
   )
+  (wire (pts (xy 60.96 44.45) (xy 60.96 46.99))
+    (stroke (width 0) (type default) (color 0 0 0 0))
+  )
   (wire (pts (xy 223.52 113.03) (xy 225.425 113.03))
     (stroke (width 0) (type default) (color 0 0 0 0))
@@
     (pin "2")
   )
-  (symbol (lib_id "Device:R") (at 60.96 47.625 0) (unit 1)
-    (in_bom yes) (on_board yes)
-    (property "Reference" "R6" (id 0) (at 62.23 45.72 0)
-      (effects (font (size 1.27 1.27)) (justify left))
-    )
-    (property "Value" "330" (id 1) (at 60.96 48.895 90)
-      (effects (font (size 1.27 1.27)) (justify left))
-    )
-    (property "Footprint" "Resistor_SMD:R_0805_2012Metric_Pad1.20x1.40mm_HandSolder" (id 2) (at 59.182 47.625 90)
-      (effects (font (size 1.27 1.27)) hide)
-    )
-    (property "Datasheet" "~" (id 3) (at 60.96 47.625 0)
-      (effects (font (size 1.27 1.27)) hide)
-    )
-    (pin "1")
-    (pin "2")
-  )
   (symbol (lib_id "power:GND") (at 153.67 191.77 0) (unit 1)
     (in_bom yes) (on_board yes) (fields_autoplaced)
@@
     (pin "2")
   )
-  (symbol (lib_id "Device:R") (at 60.96 38.1 0) (unit 1)
-    (in_bom yes) (on_board yes)
-    (property "Reference" "R5" (id 0) (at 62.23 36.195 0)
-      (effects (font (size 1.27 1.27)) (justify left))
-    )
-    (property "Value" "390" (id 1) (at 60.96 39.37 90)
-      (effects (font (size 1.27 1.27)) (justify left))
-    )
-    (property "Footprint" "Resistor_SMD:R_0805_2012Metric_Pad1.20x1.40mm_HandSolder" (id 2) (at 59.182 38.1 90)
-      (effects (font (size 1.27 1.27)) hide)
-    )
-    (property "Datasheet" "~" (id 3) (at 60.96 38.1 0)
-      (effects (font (size 1.27 1.27)) hide)
-    )
-    (pin "1")
-    (pin "2")
-  )
   (symbol (lib_id "Device:R") (at 252.73 73.025 90) (unit 1)
     (in_bom yes) (on_board yes)
@@
     (pin "1")
   )
+  (symbol (lib_id "Device:R_Potentiometer_Trim") (at 60.96 40.64 0) (unit 1)
+    (in_bom yes) (on_board yes)
+    (property "Reference" "RV?" (id 0) (at 58.42 40.64 0)
+      (effects (font (size 1.27 1.27)) (justify right))
+    )
+    (property "Value" "R_Potentiometer_Trim" (id 1) (at 58.42 41.9099 0)
+      (effects (font (size 1.27 1.27)) (justify right) hide)
+    )
+    (property "Footprint" "Potentiometer_THT:Potentiometer_Bourns_3299W_Vertical" (id 2) (at 60.96 40.64 0)
+      (effects (font (size 1.27 1.27)) hide)
+    )
+    (property "Datasheet" "~" (id 3) (at 60.96 40.64 0)
+      (effects (font (size 1.27 1.27)) hide)
+    )
+    (pin "1")
+    (pin "2")
+    (pin "3")
+  )
   (symbol (lib_id "Device:C") (at 245.11 58.42 0) (unit 1)
     (in_bom yes) (on_board yes)
@@
     (pin "2")
   )
-  (symbol (lib_id "power:GND") (at 60.96 53.975 0) (unit 1)
+  (symbol (lib_id "power:GND") (at 67.31 46.99 0) (unit 1)
     (in_bom yes) (on_board yes) (fields_autoplaced)
-    (property "Reference" "#PWR0115" (id 0) (at 60.96 60.325 0)
+    (property "Reference" "#PWR0115" (id 0) (at 67.31 53.34 0)
       (effects (font (size 1.27 1.27)) hide)
     )
-    (property "Value" "GND" (id 1) (at 60.96 58.42 0))
-    (property "Footprint" "" (id 2) (at 60.96 53.975 0)
+    (property "Value" "GND" (id 1) (at 67.31 51.435 0))
+    (property "Footprint" "" (id 2) (at 67.31 46.99 0)
       (effects (font (size 1.27 1.27)) hide)
     )
-    (property "Datasheet" "" (id 3) (at 60.96 53.975 0)
+    (property "Datasheet" "" (id 3) (at 67.31 46.99 0)
       (effects (font (size 1.27 1.27)) hide)
     )
@@
     (pin "5")
   )
+  (symbol (lib_id "power:GND") (at 60.96 46.99 0) (unit 1)
+    (in_bom yes) (on_board yes) (fields_autoplaced)
+    (property "Reference" "#PWR?" (id 0) (at 60.96 53.34 0)
+      (effects (font (size 1.27 1.27)) hide)
+    )
+    (property "Value" "GND" (id 1) (at 60.96 51.435 0))
+    (property "Footprint" "" (id 2) (at 60.96 46.99 0)
+      (effects (font (size 1.27 1.27)) hide)
+    )
+    (property "Datasheet" "" (id 3) (at 60.96 46.99 0)
+      (effects (font (size 1.27 1.27)) hide)
+    )
+    (pin "1")
+  )
   (symbol (lib_id "power:+3V3") (at 52.07 85.725 90) (unit 1)
     (in_bom yes) (on_board yes)
@@
       (reference "#PWR0166") (unit 1) (value "+3V3") (footprint "")
     )
+    (path "/7813f638-3e02-4bcc-858a-26d207714628"
+      (reference "#PWR?") (unit 1) (value "GND") (footprint "")
+    )
     (path "/5a833556-9b2d-4a89-ade5-f769671d3e3c"
       (reference "C1") (unit 1) (value "100u") (footprint "Capacitor_THT:CP_Radial_D5.0mm_P2.50mm")
@@
       (reference "R4") (unit 1) (value "100K") (footprint "Resistor_SMD:R_0805_2012Metric_Pad1.20x1.40mm_HandSolder")
     )
-    (path "/2ecb73ec-8e78-4f6a-ac11-3c758f087cf5"
-      (reference "R5") (unit 1) (value "390") (footprint "Resistor_SMD:R_0805_2012Metric_Pad1.20x1.40mm_HandSolder")
-    )
-    (path "/0a7b57aa-2b41-41f6-ab13-36c6330029bd"
-      (reference "R6") (unit 1) (value "330") (footprint "Resistor_SMD:R_0805_2012Metric_Pad1.20x1.40mm_HandSolder")
-    )
     (path "/b45802ef-f727-411f-8401-393c45e4af74"
       (reference "R7") (unit 1) (value "470") (footprint "Resistor_SMD:R_0805_2012Metric_Pad1.20x1.40mm_HandSolder")
@@
       (reference "R43") (unit 1) (value "10k") (footprint "Resistor_SMD:R_0805_2012Metric_Pad1.20x1.40mm_HandSolder")
     )
+    (path "/521a4a83-0f29-4d03-acd6-c6cd2eb7ef82"
+      (reference "RV?") (unit 1) (value "R_Potentiometer_Trim") (footprint "Potentiometer_THT:Potentiometer_Bourns_3299W_Vertical")
+    )
     (path "/8973b032-605e-4661-81d2-7c8b6490c779"

Commit message: [HDW_31] Add 1205V DC DC converter
Add of a murata NXE2S1205MC DC DC downconverter
to add 12V power supply possibility. Will maybe
not be soldered but footprints are there for
future amelioration. Helps to plug a battery
on radio
Parts:
- added J17: Conn_01x02, Connector_PinSocket_2.54mm:PinSocket_1x02_P2.54mm_Vertical, symbol Connector_Generic:Conn_01x02
- added L?: L_Coupled_1243 22n, Inductor_SMD:L_Wuerth_WE-DD-Typ-M-Typ-S, symbol Device:L_Coupled_1243
- added U2: NXE2S1205MC, Converter_DCDC:Converter_DCDC_Murata_NXExSxxxxMC_SMD, symbol Regulator_Switching:NXE2S1205MC
- gave numbers to parts that had none: 1
Connections:
- net GND: now also L?.3
- net sys_onoff_i: now also L?.2
- new net: L?.1, U2.8 (+VOUT)
- new net: L?.4, U2.7 (-VOUT)
- new net: J17.1 (Pin_1), U2.3 (+VIN)
- new net: J17.2 (Pin_2), U2.1 (-VIN)
Other:
- moved on the sheet: J6

Commit message: [HDW_36] Fixed edge cut layer
Edge.cut layer fixed with circle removed
Cleanup TICKET.md file
minor other correction
READY TO TEST. All firmware should be tested
on breadboard first before sending to production
Parts:
- added HS1: Heatsink, Heatsink:Heatsink_AAVID_TV5G_TO220_Horizontal, symbol Mechanical:Heatsink
- L1: renamed from L?; Mouser (none) -> 710-744877220
- RV1: Mouser (none) -> 652-3299W-1-102LF
Other:
- moved on the sheet: C1, C2, C3, D1, F1, J1, J17, J_pwrLed1, J_sys1, L1, R10, R8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

Commit message: Add pictures and remove epaper connector in schematics
Schematic of epaper was pointless as alone in its file. Moved to main schematic
Add pictures of schematic and PCB for documentation
Parts:
- added J13: Conn_01x08_epaper, Connector_PinSocket_2.54mm:PinSocket_1x08_P2.54mm_Vertical, symbol Connector_Generic:Conn_01x08
Connections:
- net +3V3: now also J13.1 (Pin_1)
- net EPD_BUSY: now also J13.8 (Pin_8)
- net EPD_CLK: now also J13.5 (Pin_5)
- net EPD_CS: now also J13.3 (Pin_3)
- net EPD_DC: now also J13.2 (Pin_2)
- net EPD_DIN: now also J13.6 (Pin_6)
- net EPD_RST: now also J13.7 (Pin_7)
- net GND: now also J13.4 (Pin_4)
Other:
- removed sheet btRadio_epaper

Commit message: [HDW_25] Fix mounting holes issue
Add mounting holes for screwing to radio chassis
Add mounting holes for PAM8302
Cleanup TICKETS file
Change README name
Parts:
- removed HS1: Heatsink, Heatsink:Heatsink_AAVID_TV5G_TO220_Horizontal, symbol Mechanical:Heatsink
- C4, C5, C6, C7: value 10n -> 47n
Changed lines of the file:
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@@
       (effects (font (size 1.27 1.27)) (justify left))
     )
-    (property "Value" "10n" (id 1) (at 245.11 60.833 0)
+    (property "Value" "47n" (id 1) (at 245.11 60.833 0)
       (effects (font (size 1.27 1.27)) (justify left))
     )
@@
     (pin "1")
   )
-  (symbol (lib_id "Mechanical:Heatsink") (at 59.69 22.86 0) (unit 1)
-    (in_bom yes) (on_board yes) (fields_autoplaced)
-    (property "Reference" "HS1" (id 0) (at 63.5 19.6849 0)
-      (effects (font (size 1.27 1.27)) (justify left))
-    )
-    (property "Value" "Heatsink" (id 1) (at 63.5 22.2249 0)
-      (effects (font (size 1.27 1.27)) (justify left))
-    )
-    (property "Footprint" "Heatsink:Heatsink_AAVID_TV5G_TO220_Horizontal" (id 2) (at 59.9948 22.86 0)
-      (effects (font (size 1.27 1.27)) hide)
-    )
-    (property "Datasheet" "~" (id 3) (at 59.9948 22.86 0)
-      (effects (font (size 1.27 1.27)) hide)
-    )
-  )
   (symbol (lib_id "Connector_Generic:Conn_01x02") (at 101.6 24.13 270) (mirror x) (unit 1)
     (in_bom yes) (on_board yes)
@@
       (effects (font (size 1.27 1.27)) (justify left))
     )
-    (property "Value" "10n" (id 1) (at 245.11 83.693 0)
+    (property "Value" "47n" (id 1) (at 245.11 83.693 0)
       (effects (font (size 1.27 1.27)) (justify left))
     )
@@
       (effects (font (size 1.27 1.27)) (justify left))
     )
-    (property "Value" "10n" (id 1) (at 239.395 60.833 0)
+    (property "Value" "47n" (id 1) (at 239.395 60.833 0)
       (effects (font (size 1.27 1.27)) (justify left))
     )
@@
       (effects (font (size 1.27 1.27)) (justify left))
     )
-    (property "Value" "10n" (id 1) (at 239.395 83.693 0)
+    (property "Value" "47n" (id 1) (at 239.395 83.693 0)
       (effects (font (size 1.27 1.27)) (justify left))
     )
@@
     )
     (path "/9d5daadc-2c65-4e73-9d00-62b7fee36ca1"
-      (reference "C4") (unit 1) (value "10n") (footprint "Resistor_SMD:R_0805_2012Metric_Pad1.20x1.40mm_HandSolder")
+      (reference "C4") (unit 1) (value "47n") (footprint "Resistor_SMD:R_0805_2012Metric_Pad1.20x1.40mm_HandSolder")
     )
     (path "/d602545a-8177-4f7e-8ff5-63bcc0c7892b"
-      (reference "C5") (unit 1) (value "10n") (footprint "Resistor_SMD:R_0805_2012Metric_Pad1.20x1.40mm_HandSolder")
+      (reference "C5") (unit 1) (value "47n") (footprint "Resistor_SMD:R_0805_2012Metric_Pad1.20x1.40mm_HandSolder")
     )
     (path "/54655d78-8059-441c-920a-420752329d40"
-      (reference "C6") (unit 1) (value "10n") (footprint "Resistor_SMD:R_0805_2012Metric_Pad1.20x1.40mm_HandSolder")
+      (reference "C6") (unit 1) (value "47n") (footprint "Resistor_SMD:R_0805_2012Metric_Pad1.20x1.40mm_HandSolder")
     )
     (path "/6cb65816-3452-4e9d-813f-a1607f88004a"
-      (reference "C7") (unit 1) (value "10n") (footprint "Resistor_SMD:R_0805_2012Metric_Pad1.20x1.40mm_HandSolder")
+      (reference "C7") (unit 1) (value "47n") (footprint "Resistor_SMD:R_0805_2012Metric_Pad1.20x1.40mm_HandSolder")
     )
     (path "/93984d3e-1049-40c4-85f7-3f9031f77d6e/1aa40ec2-1492-4818-adc7-88e45d293bd1"
@@
       (reference "F1") (unit 1) (value "Polyfuse 1,5A") (footprint "Fuse:Fuse_BelFuse_0ZRE0005FF_L8.3mm_W3.8mm")
     )
-    (path "/5add5888-0723-45e1-a8e0-e7baac28fb38"
-      (reference "HS1") (unit 1) (value "Heatsink") (footprint "Heatsink:Heatsink_AAVID_TV5G_TO220_Horizontal")
-    )
     (path "/8d89841f-5f2d-4255-9b3d-fcb2b5092c11"

Commit message: [HDW_37] Add files for production
Add JLCPCB form BOM and own format BOM for mouser ref tracking
Minor correction on schematic: J16 -> J_VIII1
Parts:
- R1, R2, R3, R4: value 100K -> 100k
Changed lines of the file:
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@@
       (effects (font (size 1.27 1.27)) (justify left))
     )
-    (property "Value" "100K" (id 1) (at 43.815 114.3 90)
+    (property "Value" "100k" (id 1) (at 43.815 114.3 90)
       (effects (font (size 1.27 1.27)) (justify left))
     )
@@
       (effects (font (size 1.27 1.27)) (justify left))
     )
-    (property "Value" "100K" (id 1) (at 43.815 129.54 90)
+    (property "Value" "100k" (id 1) (at 43.815 129.54 90)
       (effects (font (size 1.27 1.27)) (justify left))
     )
@@
       (effects (font (size 1.27 1.27)) (justify left))
     )
-    (property "Value" "100K" (id 1) (at 28.575 129.54 90)
+    (property "Value" "100k" (id 1) (at 28.575 129.54 90)
       (effects (font (size 1.27 1.27)) (justify left))
     )
@@
       (effects (font (size 1.27 1.27)) (justify left))
     )
-    (property "Value" "100K" (id 1) (at 28.575 114.3 90)
+    (property "Value" "100k" (id 1) (at 28.575 114.3 90)
       (effects (font (size 1.27 1.27)) (justify left))
     )
@@
       (reference "J15") (unit 1) (value "Conn_01x02_classD_SD") (footprint "Connector_PinSocket_2.54mm:PinSocket_1x02_P2.54mm_Vertical")
     )
-    (path "/f502a33a-d5e4-4b91-95a6-ac6a3abcb73b/8032c36b-408e-4af8-a36d-abf19ffbabfb"
-      (reference "J16") (unit 1) (value "Conn_02x12_Odd_Even") (footprint "Connector_PinSocket_2.54mm:PinSocket_2x12_P2.54mm_Vertical")
-    )
     (path "/768586d6-e9e8-47f1-8c19-5a1ef24ed007"
       (reference "J17") (unit 1) (value "Conn_01x02") (footprint "Connector_PinSocket_2.54mm:PinSocket_1x02_P2.54mm_Vertical")
@@
       (reference "J_VII1") (unit 1) (value "Conn_02x03_Odd_Even") (footprint "Connector_PinSocket_2.54mm:PinSocket_2x03_P2.54mm_Vertical")
     )
+    (path "/f502a33a-d5e4-4b91-95a6-ac6a3abcb73b/8032c36b-408e-4af8-a36d-abf19ffbabfb"
+      (reference "J_VIII1") (unit 1) (value "Conn_02x12_Odd_Even") (footprint "Connector_PinSocket_2.54mm:PinSocket_2x12_P2.54mm_Vertical")
+    )
     (path "/f502a33a-d5e4-4b91-95a6-ac6a3abcb73b/f7779aac-997c-4344-b3b4-52eb8625f4c4"
       (reference "J_X1") (unit 1) (value "Conn_02x09_Odd_Even") (footprint "Connector_PinSocket_2.54mm:PinSocket_2x09_P2.54mm_Vertical")
@@
     )
     (path "/eeb0776d-6559-4b91-9fc8-59c644c43ea6"
-      (reference "R1") (unit 1) (value "100K") (footprint "Resistor_SMD:R_0805_2012Metric_Pad1.20x1.40mm_HandSolder")
+      (reference "R1") (unit 1) (value "100k") (footprint "Resistor_SMD:R_0805_2012Metric_Pad1.20x1.40mm_HandSolder")
     )
     (path "/c785185a-671a-42dc-9104-67f88f7b72f9"
-      (reference "R2") (unit 1) (value "100K") (footprint "Resistor_SMD:R_0805_2012Metric_Pad1.20x1.40mm_HandSolder")
+      (reference "R2") (unit 1) (value "100k") (footprint "Resistor_SMD:R_0805_2012Metric_Pad1.20x1.40mm_HandSolder")
     )
     (path "/09a54c94-673c-4aa0-9deb-5558bd66f008"
-      (reference "R3") (unit 1) (value "100K") (footprint "Resistor_SMD:R_0805_2012Metric_Pad1.20x1.40mm_HandSolder")
+      (reference "R3") (unit 1) (value "100k") (footprint "Resistor_SMD:R_0805_2012Metric_Pad1.20x1.40mm_HandSolder")
     )
     (path "/b3025289-cffc-4ff1-9309-bd041a277055"
-      (reference "R4") (unit 1) (value "100K") (footprint "Resistor_SMD:R_0805_2012Metric_Pad1.20x1.40mm_HandSolder")
+      (reference "R4") (unit 1) (value "100k") (footprint "Resistor_SMD:R_0805_2012Metric_Pad1.20x1.40mm_HandSolder")
     )
     (path "/b45802ef-f727-411f-8401-393c45e4af74"

Commit message: [HDW_38] Fix Bt communication wires
Bluetooth Rx pin connected to GPIO4 of RP240
Bluetooth Tx pin connected to GPIO5 of RP2040
Connections:
- net BT_UART_RX: now also JRP4020L_1.6 (Pin_6); no longer JRP4020L_1.4 (Pin_4)
- net BT_UART_TX: now also JRP4020L_1.7 (Pin_7); no longer JRP4020L_1.5 (Pin_5)
- net FM_RST: now also JRP4020L_1.4 (Pin_4); no longer JRP4020L_1.6 (Pin_6)
- net FM_SEN: now also JRP4020L_1.5 (Pin_5); no longer JRP4020L_1.7 (Pin_7)
Changed lines of the file:
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@@
+    )
+  )
+  (global_label "BT_UART_RX" (shape input) (at 223.52 113.03 180) (fields_autoplaced)
+    (effects (font (size 1.27 1.27)) (justify right))
+    (property "Intersheet References" "${INTERSHEET_REFS}" (id 0) (at 209.7979 112.9506 0)
+      (effects (font (size 1.27 1.27)) (justify right) hide)
     )
   )
@@
     )
   )
-  (global_label "BT_UART_RX" (shape input) (at 223.52 107.95 180) (fields_autoplaced)
-    (effects (font (size 1.27 1.27)) (justify right))
-    (property "Intersheet References" "${INTERSHEET_REFS}" (id 0) (at 209.7979 107.8706 0)
+  (global_label "FM_SEN" (shape input) (at 223.52 110.49 180) (fields_autoplaced)
+    (effects (font (size 1.27 1.27)) (justify right))
+    (property "Intersheet References" "${INTERSHEET_REFS}" (id 0) (at 213.9102 110.4106 0)
+      (effects (font (size 1.27 1.27)) (justify right) hide)
+    )
+  )
+  (global_label "FM_RST" (shape input) (at 223.52 107.95 180) (fields_autoplaced)
+    (effects (font (size 1.27 1.27)) (justify right))
+    (property "Intersheet References" "${INTERSHEET_REFS}" (id 0) (at 214.1521 107.8706 0)
       (effects (font (size 1.27 1.27)) (justify right) hide)
     )
@@
     )
   )
-  (global_label "FM_RST" (shape input) (at 223.52 113.03 180) (fields_autoplaced)
-    (effects (font (size 1.27 1.27)) (justify right))
-    (property "Intersheet References" "${INTERSHEET_REFS}" (id 0) (at 214.1521 112.9506 0)
-      (effects (font (size 1.27 1.27)) (justify right) hide)
-    )
-  )
   (global_label "BT_PWREN" (shape input) (at 40.005 188.595 180) (fields_autoplaced)
     (effects (font (size 1.27 1.27)) (justify right))
@@
     )
   )
-  (global_label "FM_SEN" (shape input) (at 223.52 115.57 180) (fields_autoplaced)
-    (effects (font (size 1.27 1.27)) (justify right))
-    (property "Intersheet References" "${INTERSHEET_REFS}" (id 0) (at 213.9102 115.4906 0)
-      (effects (font (size 1.27 1.27)) (justify right) hide)
-    )
-  )
   (global_label "BT_MIC_R+" (shape input) (at 59.69 158.115 0) (fields_autoplaced)
     (effects (font (size 1.27 1.27)) (justify left))
@@
     )
   )
+  (global_label "BT_UART_TX" (shape input) (at 223.52 115.57 180) (fields_autoplaced)
+    (effects (font (size 1.27 1.27)) (justify right))
+    (property "Intersheet References" "${INTERSHEET_REFS}" (id 0) (at 210.1002 115.4906 0)
+      (effects (font (size 1.27 1.27)) (justify right) hide)
+    )
+  )
   (global_label "BT_SPI_SCK" (shape input) (at 59.69 173.355 0) (fields_autoplaced)
     (effects (font (size 1.27 1.27)) (justify left))
@@
       (effects (font (size 1.27 1.27)) (justify right) hide)
     )
-  )
-  (global_label "BT_UART_TX" (shape input) (at 223.52 110.49 180) (fields_autoplaced)
-    (effects (font (size 1.27 1.27)) (justify right))
-    (property "Intersheet References" "${INTERSHEET_REFS}" (id 0) (at 210.1002 110.4106 0)
-      (effects (font (size 1.27 1.27)) (justify right) hide)
-    )
