File: 03_Development/Hardware/Proto_Bluetooth/Board_Bluetooth_radio_platform.kicad_sch (KiCad schematic)
At the start: 51 parts, among them J1 Conn_01x02, J10 Conn_01x03, J11 HMI_rotaryEncoder_1, J12 HMI_rotaryEncoder_1, J13 Conn_01x08_epaper, J17 Conn_01x02, J19 Conn_01x02_rn52_usb, J2 Conn_01x08, J3 BT_RN52_connector_left, J4 Conn_01x02, J5 BT_RN52_connector_right, J6 FM_interface, J7 BT_debug_connector, J8 BT_extension_connector, J9 SYS_debug_connector, SW1 SW_Push, U1 LM317_TO-220, U2 NXE2S1205MC

Commit message: [HDW_39] Fix pull ups and pull down resistances
RP2040 internal's pull up/down are actually 80 kOhms
which is quite few. ALl filters and external pull up-down
are too high for them and incoming signal on RP2040
is too small.
Set all to either 4.7 kOhms or 10 kOhms
Parts:
- C4, C5, C6, C7: value 47n -> 10n
- R1, R11, R12, R2, R3, R4: value 100k -> 10k
- R13, R14, R15, R16: value 470k -> 10k

Commit message: [HDW_41] FIX communication lines to central unit
FM, EP and BT modules had been routed to ports of RP2040 which don't allow
UART or I2C and must have been changed
Connections:
- net BT_UART_RX: now also JRP4020L_1.11 (Pin_11); no longer JRP4020L_1.6 (Pin_6)
- net BT_UART_TX: now also JRP4020L_1.12 (Pin_12); no longer JRP4020L_1.7 (Pin_7)
- net EPD_CS: now also JRP4020L_1.20 (Pin_20); no longer JRP4020L_1.12 (Pin_12)
- net EPD_DC: now also JRP4020L_1.19 (Pin_19); no longer JRP4020L_1.11 (Pin_11)
- net FM_GPIO1: now also JRP4020L_1.10 (Pin_10); no longer JRP4020L_1.20 (Pin_20)
- net FM_GPIO2: now also JRP4020L_1.9 (Pin_9); no longer JRP4020L_1.19 (Pin_19)
- net FM_SCLK: now also JRP4020L_1.7 (Pin_7); no longer JRP4020L_1.10 (Pin_10)
- net FM_SDIO: now also JRP4020L_1.6 (Pin_6); no longer JRP4020L_1.9 (Pin_9)
Changed lines of the file:
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@@
     (stroke (width 0) (type default) (color 0 0 0 0))
   )
-  (wire (pts (xy 224.155 146.05) (xy 225.425 146.05))
+  (wire (pts (xy 223.52 146.05) (xy 225.425 146.05))
     (stroke (width 0) (type default) (color 0 0 0 0))
   )
@@
     (stroke (width 0) (type default) (color 0 0 0 0))
   )
-  (wire (pts (xy 224.155 148.59) (xy 225.425 148.59))
+  (wire (pts (xy 223.52 148.59) (xy 225.425 148.59))
     (stroke (width 0) (type default) (color 0 0 0 0))
   )
@@
     (stroke (width 0) (type default) (color 0 0 0 0))
   )
+  (global_label "BT_UART_RX" (shape input) (at 223.52 125.73 180) (fields_autoplaced)
+    (effects (font (size 1.27 1.27)) (justify right))
+    (property "Intersheet References" "${INTERSHEET_REFS}" (id 0) (at 209.7979 125.6506 0)
+      (effects (font (size 1.27 1.27)) (justify right) hide)
+    )
+  )
   (global_label "BT_SPI_SS" (shape input) (at 59.69 178.435 0) (fields_autoplaced)
     (effects (font (size 1.27 1.27)) (justify left))
@@
     )
   )
-  (global_label "BT_UART_RX" (shape input) (at 223.52 113.03 180) (fields_autoplaced)
-    (effects (font (size 1.27 1.27)) (justify right))
-    (property "Intersheet References" "${INTERSHEET_REFS}" (id 0) (at 209.7979 112.9506 0)
-      (effects (font (size 1.27 1.27)) (justify right) hide)
-    )
-  )
   (global_label "FM_SDIO" (shape input) (at 91.44 182.88 180) (fields_autoplaced)
     (effects (font (size 1.27 1.27)) (justify right))
@@
     )
   )
+  (global_label "FM_GPIO1" (shape input) (at 223.52 123.19 180) (fields_autoplaced)
+    (effects (font (size 1.27 1.27)) (justify right))
+    (property "Intersheet References" "${INTERSHEET_REFS}" (id 0) (at 211.9145 123.1106 0)
+      (effects (font (size 1.27 1.27)) (justify right) hide)
+    )
+  )
   (global_label "sys_3V3_EN" (shape input) (at 254 107.95 0) (fields_autoplaced)
     (effects (font (size 1.27 1.27)) (justify left))
@@
     )
   )
-  (global_label "EPD_DC" (shape input) (at 223.52 125.73 180) (fields_autoplaced)
-    (effects (font (size 1.27 1.27)) (justify right))
-    (property "Intersheet References" "${INTERSHEET_REFS}" (id 0) (at 213.9102 125.6506 0)
-      (effects (font (size 1.27 1.27)) (justify right) hide)
-    )
-  )
   (global_label "BT_SPKR_R+" (shape input) (at 59.944 145.415 0) (fields_autoplaced)
     (effects (font (size 1.27 1.27)) (justify left))
@@
     )
   )
-  (global_label "EPD_CS" (shape input) (at 223.52 128.27 180) (fields_autoplaced)
-    (effects (font (size 1.27 1.27)) (justify right))
-    (property "Intersheet References" "${INTERSHEET_REFS}" (id 0) (at 213.9707 128.1906 0)
-      (effects (font (size 1.27 1.27)) (justify right) hide)
-    )
-  )
   (global_label "DBG_RST" (shape input) (at 252.73 125.73 0) (fields_autoplaced)
     (effects (font (size 1.27 1.27)) (justify left))
@@
     )
   )
-  (global_label "FM_GPIO1" (shape input) (at 224.155 148.59 180) (fields_autoplaced)
-    (effects (font (size 1.27 1.27)) (justify right))
-    (property "Intersheet References" "${INTERSHEET_REFS}" (id 0) (at 212.5495 148.5106 0)
-      (effects (font (size 1.27 1.27)) (justify right) hide)
-    )
-  )
   (global_label "FM_GPIO2" (shape input) (at 91.44 170.18 180) (fields_autoplaced)
     (effects (font (size 1.27 1.27)) (justify right))
@@
     )
   )
-  (global_label "FM_SDIO" (shape input) (at 223.52 120.65 180) (fields_autoplaced)
-    (effects (font (size 1.27 1.27)) (justify right))
-    (property "Intersheet References" "${INTERSHEET_REFS}" (id 0) (at 213.1845 120.5706 0)
-      (effects (font (size 1.27 1.27)) (justify right) hide)
-    )
-  )
   (global_label "DBG_SWCLK" (shape input) (at 134.62 186.69 180) (fields_autoplaced)
     (effects (font (size 1.27 1.27)) (justify right))
@@
     )
   )
+  (global_label "FM_GPIO2" (shape input) (at 223.52 120.65 180) (fields_autoplaced)
+    (effects (font (size 1.27 1.27)) (justify right))
+    (property "Intersheet References" "${INTERSHEET_REFS}" (id 0) (at 211.9145 120.5706 0)
+      (effects (font (size 1.27 1.27)) (justify right) hide)
+    )
+  )
   (global_label "BT_MIC_R+" (shape input) (at 59.69 158.115 0) (fields_autoplaced)
     (effects (font (size 1.27 1.27)) (justify left))
@@
     )
   )
+  (global_label "EPD_DC" (shape input) (at 223.52 146.05 180) (fields_autoplaced)
+    (effects (font (size 1.27 1.27)) (justify right))
+    (property "Intersheet References" "${INTERSHEET_REFS}" (id 0) (at 213.9102 145.9706 0)
+      (effects (font (size 1.27 1.27)) (justify right) hide)
+    )
+  )
+  (global_label "FM_SCLK" (shape input) (at 223.52 115.57 180) (fields_autoplaced)
+    (effects (font (size 1.27 1.27)) (justify right))
+    (property "Intersheet References" "${INTERSHEET_REFS}" (id 0) (at 212.8217 115.4906 0)
+      (effects (font (size 1.27 1.27)) (justify right) hide)
+    )
+  )
   (global_label "BT_GPIO6" (shape input) (at 135.89 165.1 180) (fields_autoplaced)
     (effects (font (size 1.27 1.27)) (justify right))
@@
     )
   )
-  (global_label "FM_SCLK" (shape input) (at 223.52 123.19 180) (fields_autoplaced)
-    (effects (font (size 1.27 1.27)) (justify right))
-    (property "Intersheet References" "${INTERSHEET_REFS}" (id 0) (at 212.8217 123.1106 0)
-      (effects (font (size 1.27 1.27)) (justify right) hide)
-    )
-  )
   (global_label "DBG_UART_RX" (shape input) (at 150.495 181.61 0) (fields_autoplaced)
     (effects (font (size 1.27 1.27)) (justify left))
@@
     )
   )
-  (global_label "BT_UART_TX" (shape input) (at 223.52 115.57 180) (fields_autoplaced)
-    (effects (font (size 1.27 1.27)) (justify right))
-    (property "Intersheet References" "${INTERSHEET_REFS}" (id 0) (at 210.1002 115.4906 0)
-      (effects (font (size 1.27 1.27)) (justify right) hide)
-    )
-  )
   (global_label "BT_SPI_SCK" (shape input) (at 59.69 173.355 0) (fields_autoplaced)
     (effects (font (size 1.27 1.27)) (justify left))
@@
     )
   )
+  (global_label "FM_SDIO" (shape input) (at 223.52 113.03 180) (fields_autoplaced)
+    (effects (font (size 1.27 1.27)) (justify right))
+    (property "Intersheet References" "${INTERSHEET_REFS}" (id 0) (at 213.1845 112.9506 0)
+      (effects (font (size 1.27 1.27)) (justify right) hide)
+    )
+  )
   (global_label "BT_GPIO2" (shape input) (at 39.37 145.415 180) (fields_autoplaced)
     (effects (font (size 1.27 1.27)) (justify right))
@@
     )
   )
+  (global_label "EPD_CS" (shape input) (at 223.52 148.59 180) (fields_autoplaced)
+    (effects (font (size 1.27 1.27)) (justify right))
+    (property "Intersheet References" "${INTERSHEET_REFS}" (id 0) (at 213.9707 148.5106 0)
+      (effects (font (size 1.27 1.27)) (justify right) hide)
+    )
+  )
   (global_label "SYS_audio_sw" (shape input) (at 252.73 128.27 0) (fields_autoplaced)
     (effects (font (size 1.27 1.27)) (justify left))
@@
     )
   )
-  (global_label "FM_GPIO2" (shape input) (at 224.155 146.05 180) (fields_autoplaced)
-    (effects (font (size 1.27 1.27)) (justify right))
-    (property "Intersheet References" "${INTERSHEET_REFS}" (id 0) (at 212.5495 145.9706 0)
-      (effects (font (size 1.27 1.27)) (justify right) hide)
-    )
-  )
   (global_label "BT_UART_RTS" (shape input) (at 39.878 173.355 180) (fields_autoplaced)
     (effects (font (size 1.27 1.27)) (justify right))
@@
       (effects (font (size 1.27 1.27)) (justify right) hide)
     )
+  )
+  (global_label "BT_UART_TX" (shape input) (at 223.52 128.27 180) (fields_autoplaced)
+    (effects (font (size 1.27 1.27)) (justify right))
+    (property "Intersheet References" "${INTERSHEET_REFS}" (id 0) (at 210.1002 128.1906 0)
+      (effects (font (size 1.27 1.27)) (justify right) hide)
+    )

Commit message: [HDW_45] FIX remove of 12V power supply
Parts:
- removed J17: Conn_01x02, Connector_PinSocket_2.54mm:PinSocket_1x02_P2.54mm_Vertical, symbol Connector_Generic:Conn_01x02
- removed L1: L_Coupled_1243 22n, Inductor_SMD:L_Wuerth_WE-DD-Typ-M-Typ-S, symbol Device:L_Coupled_1243
- removed U2: NXE2S1205MC, Converter_DCDC:Converter_DCDC_Murata_NXExSxxxxMC_SMD, symbol Regulator_Switching:NXE2S1205MC
Changed lines of the file:
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@@
     (stroke (width 0) (type default) (color 0 0 0 0))
   )
-  (wire (pts (xy 52.07 73.66) (xy 50.8 73.66))
-    (stroke (width 0) (type default) (color 0 0 0 0))
-  )
   (wire (pts (xy 57.785 147.955) (xy 59.944 147.955))
     (stroke (width 0) (type default) (color 0 0 0 0))
   )
-  (wire (pts (xy 52.07 63.5) (xy 50.8 63.5))
-    (stroke (width 0) (type default) (color 0 0 0 0))
-  )
   (wire (pts (xy 48.133 119.38) (xy 48.133 121.412))
     (stroke (width 0) (type default) (color 0 0 0 0))
@@
     (stroke (width 0) (type default) (color 0 0 0 0))
   )
-  (wire (pts (xy 63.5 66.04) (xy 66.04 66.04))
-    (stroke (width 0) (type default) (color 0 0 0 0))
-  )
   (wire (pts (xy 137.16 78.105) (xy 141.605 78.105))
     (stroke (width 0) (type default) (color 0 0 0 0))
@@
     (stroke (width 0) (type default) (color 0 0 0 0))
   )
-  (wire (pts (xy 66.04 73.66) (xy 66.04 71.12))
-    (stroke (width 0) (type default) (color 0 0 0 0))
-  )
   (wire (pts (xy 261.62 25.4) (xy 264.16 25.4))
     (stroke (width 0) (type default) (color 0 0 0 0))
@@
     (stroke (width 0) (type default) (color 0 0 0 0))
   )
-  (wire (pts (xy 52.07 66.04) (xy 52.07 63.5))
-    (stroke (width 0) (type default) (color 0 0 0 0))
-  )
   (wire (pts (xy 28.575 121.92) (xy 27.305 121.92))
     (stroke (width 0) (type default) (color 0 0 0 0))
@@
     (stroke (width 0) (type default) (color 0 0 0 0))
   )
-  (wire (pts (xy 22.86 67.31) (xy 22.86 63.5))
-    (stroke (width 0) (type default) (color 0 0 0 0))
-  )
   (wire (pts (xy 95.25 180.34) (xy 91.44 180.34))
     (stroke (width 0) (type default) (color 0 0 0 0))
@@
     (stroke (width 0) (type default) (color 0 0 0 0))
   )
-  (wire (pts (xy 21.59 69.85) (xy 22.86 69.85))
-    (stroke (width 0) (type default) (color 0 0 0 0))
-  )
   (wire (pts (xy 59.69 36.83) (xy 59.69 38.735))
     (stroke (width 0) (type default) (color 0 0 0 0))
   )
-  (wire (pts (xy 21.59 67.31) (xy 22.86 67.31))
-    (stroke (width 0) (type default) (color 0 0 0 0))
-  )
   (wire (pts (xy 154.94 139.7) (xy 154.94 144.78))
     (stroke (width 0) (type default) (color 0 0 0 0))
@@
     (stroke (width 0) (type default) (color 0 0 0 0))
   )
-  (wire (pts (xy 22.86 69.85) (xy 22.86 73.66))
-    (stroke (width 0) (type default) (color 0 0 0 0))
-  )
   (wire (pts (xy 43.815 106.045) (xy 43.815 107.95))
     (stroke (width 0) (type default) (color 0 0 0 0))
@@
     (stroke (width 0) (type default) (color 0 0 0 0))
   )
-  (wire (pts (xy 66.04 71.12) (xy 63.5 71.12))
-    (stroke (width 0) (type default) (color 0 0 0 0))
-  )
   (wire (pts (xy 69.85 106.045) (xy 69.85 107.315))
     (stroke (width 0) (type default) (color 0 0 0 0))
@@
     (stroke (width 0) (type default) (color 0 0 0 0))
   )
-  (wire (pts (xy 22.86 73.66) (xy 25.4 73.66))
-    (stroke (width 0) (type default) (color 0 0 0 0))
-  )
   (wire (pts (xy 135.89 162.56) (xy 137.795 162.56))
     (stroke (width 0) (type default) (color 0 0 0 0))
@@
     (stroke (width 0) (type default) (color 0 0 0 0))
   )
-  (wire (pts (xy 53.34 71.12) (xy 52.07 71.12))
-    (stroke (width 0) (type default) (color 0 0 0 0))
-  )
   (wire (pts (xy 245.11 70.485) (xy 245.11 77.47))
     (stroke (width 0) (type default) (color 0 0 0 0))
@@
     (stroke (width 0) (type default) (color 0 0 0 0))
   )
-  (wire (pts (xy 52.07 71.12) (xy 52.07 73.66))
-    (stroke (width 0) (type default) (color 0 0 0 0))
-  )
   (wire (pts (xy 235.585 75.565) (xy 251.46 75.565))
     (stroke (width 0) (type default) (color 0 0 0 0))
@@
     (stroke (width 0) (type default) (color 0 0 0 0))
   )
-  (wire (pts (xy 53.34 66.04) (xy 52.07 66.04))
-    (stroke (width 0) (type default) (color 0 0 0 0))
-  )
   (wire (pts (xy 251.46 85.09) (xy 251.46 86.995))
     (stroke (width 0) (type default) (color 0 0 0 0))
@@
     (stroke (width 0) (type default) (color 0 0 0 0))
   )
-  (wire (pts (xy 22.86 63.5) (xy 25.4 63.5))
-    (stroke (width 0) (type default) (color 0 0 0 0))
-  )
   (wire (pts (xy 223.52 135.89) (xy 225.425 135.89))
     (stroke (width 0) (type default) (color 0 0 0 0))
@@
     )
   )
-  (global_label "sys_onoff_i" (shape input) (at 66.04 66.04 0) (fields_autoplaced)
-    (effects (font (size 1.27 1.27)) (justify left))
-    (property "Intersheet References" "${INTERSHEET_REFS}" (id 0) (at 78.9155 65.9606 0)
-      (effects (font (size 1.27 1.27)) (justify left) hide)
-    )
-  )
   (global_label "RE1_A" (shape input) (at 252.73 140.97 0) (fields_autoplaced)
     (effects (font (size 1.27 1.27)) (justify left))
@@
     (pin "1")
   )
-  (symbol (lib_id "Device:L_Coupled_1243") (at 58.42 68.58 0) (unit 1)
-    (in_bom yes) (on_board yes)
-    (property "Reference" "L1" (id 0) (at 58.42 64.77 0))
-    (property "Value" "L_Coupled_1243 22n" (id 1) (at 58.039 63.5 0)
-      (effects (font (size 1.27 1.27)) hide)
-    )
-    (property "Footprint" "Inductor_SMD:L_Wuerth_WE-DD-Typ-M-Typ-S" (id 2) (at 58.42 68.58 0)
-      (effects (font (size 1.27 1.27)) hide)
-    )
-    (property "Datasheet" "" (id 3) (at 58.42 68.58 0)
-      (effects (font (size 1.27 1.27)) hide)
-    )
-    (property "Mouser" "710-744877220 " (id 4) (at 58.42 68.58 0)
-      (effects (font (size 1.27 1.27)) hide)
-    )
-    (pin "1")
-    (pin "2")
-    (pin "3")
-    (pin "4")
-  )
   (symbol (lib_id "Device:R") (at 252.73 70.485 90) (unit 1)
     (in_bom yes) (on_board yes)
@@
     (pin "2")
   )
-  (symbol (lib_id "power:GND") (at 66.04 73.66 0) (unit 1)
-    (in_bom yes) (on_board yes) (fields_autoplaced)
-    (property "Reference" "#PWR06" (id 0) (at 66.04 80.01 0)
-      (effects (font (size 1.27 1.27)) hide)
-    )
-    (property "Value" "GND" (id 1) (at 66.04 78.105 0))
-    (property "Footprint" "" (id 2) (at 66.04 73.66 0)
-      (effects (font (size 1.27 1.27)) hide)
-    )
-    (property "Datasheet" "" (id 3) (at 66.04 73.66 0)
-      (effects (font (size 1.27 1.27)) hide)
-    )
-    (pin "1")
-  )
   (symbol (lib_id "power:GND") (at 43.815 132.08 0) (unit 1)
     (in_bom yes) (on_board yes) (fields_autoplaced)
@@
     (pin "1")
   )
-  (symbol (lib_id "Connector_Generic:Conn_01x02") (at 16.51 67.31 0) (mirror y) (unit 1)
-    (in_bom yes) (on_board yes)
-    (property "Reference" "J17" (id 0) (at 16.51 64.77 0))
-    (property "Value" "Conn_01x02" (id 1) (at 16.51 74.295 0)
-      (effects (font (size 1.27 1.27)) hide)
-    )
-    (property "Footprint" "Connector_PinSocket_2.54mm:PinSocket_1x02_P2.54mm_Vertical" (id 2) (at 16.51 67.31 0)
-      (effects (font (size 1.27 1.27)) hide)
-    )
-    (property "Datasheet" "~" (id 3) (at 16.51 67.31 0)
-      (effects (font (size 1.27 1.27)) hide)
-    )
-    (pin "1")
-    (pin "2")
-  )
   (symbol (lib_id "Connector_Generic:Conn_01x05") (at 269.24 75.565 0) (unit 1)
     (in_bom yes) (on_board yes) (fields_autoplaced)
@@
     (pin "1")
   )
-  (symbol (lib_id "Regulator_Switching:NXE2S1205MC") (at 38.1 68.58 0) (unit 1)
-    (in_bom yes) (on_board yes)
-    (property "Reference" "U2" (id 0) (at 38.1 58.42 0))
-    (property "Value" "NXE2S1205MC" (id 1) (at 38.1 58.42 0)
-      (effects (font (size 1.27 1.27)) hide)
-    )
-    (property "Footprint" "Converter_DCDC:Converter_DCDC_Murata_NXExSxxxxMC_SMD" (id 2) (at 38.1 77.47 0)
-      (effects (font (size 1.27 1.27)) hide)
-    )
-    (property "Datasheet" "https://www.murata.com/products/productdata/8807031898142/kdc-nxe2.pdf" (id 3) (at 38.1 81.28 0)
-      (effects (font (size 1.27 1.27)) hide)
-    )
-    (pin "1")
-    (pin "14")
-    (pin "3")
-    (pin "7")
-    (pin "8")
-  )
   (symbol (lib_id "Device:R") (at 252.73 47.625 90) (unit 1)
     (in_bom yes) (on_board yes)
@@
       (reference "#PWR05") (unit 1) (value "+3V3") (footprint "")
     )
-    (path "/4c2395b1-93f0-4773-9050-c9b491222585"
-      (reference "#PWR06") (unit 1) (value "GND") (footprint "")
-    )
     (path "/42059c44-b96f-4aea-b8b2-233d1cdc091d"
       (reference "#PWR07") (unit 1) (value "GND") (footprint "")
@@
       (reference "J15") (unit 1) (value "Conn_01x02_classD_SD") (footprint "Connector_PinSocket_2.54mm:PinSocket_1x02_P2.54mm_Vertical")
     )
-    (path "/768586d6-e9e8-47f1-8c19-5a1ef24ed007"
-      (reference "J17") (unit 1) (value "Conn_01x02") (footprint "Connector_PinSocket_2.54mm:PinSocket_1x02_P2.54mm_Vertical")
-    )
     (path "/2e24ea67-ad62-48bc-ab1f-15a6212df5eb"
       (reference "J19") (unit 1) (value "Conn_01x02_rn52_usb") (footprint "Connector_PinHeader_2.54mm:PinHeader_1x02_P2.54mm_Vertical")
@@
       (reference "J_sys1") (unit 1) (value "Conn_01x02") (footprint "Connector_PinSocket_2.54mm:PinSocket_1x02_P2.54mm_Vertical")
     )
-    (path "/48208bc4-e2ab-4270-bf91-3f3e4baaa20b"
-      (reference "L1") (unit 1) (value "L_Coupled_1243 22n") (footprint "Inductor_SMD:L_Wuerth_WE-DD-Typ-M-Typ-S")
-    )
     (path "/eeb0776d-6559-4b91-9fc8-59c644c43ea6"
       (reference "R1") (unit 1) (value "10k") (footprint "Resistor_SMD:R_0805_2012Metric_Pad1.20x1.40mm_HandSolder")
@@
       (reference "U1") (unit 1) (value "LM317_TO-220") (footprint "Package_TO_SOT_THT:TO-220-3_Horizontal_TabDown")
     )
-    (path "/f6d28571-1404-44c5-86fb-5b9a06497f09"
-      (reference "U2") (unit 1) (value "NXE2S1205MC") (footprint "Converter_DCDC:Converter_DCDC_Murata_NXExSxxxxMC_SMD")
-    )
     (path "/93984d3e-1049-40c4-85f7-3f9031f77d6e/2c8a87db-3d29-497c-8252-401310edddce"

Commit message: [HDW_49] FIX place of elements for new version
Remove micro i/o from RN52 as they won't be used
Move power supply down on PCB
Move class D amplifier
Add hole for push buttons mounting
Parts:
- removed J8: BT_extension_connector, Connector_PinSocket_2.54mm:PinSocket_2x08_P2.54mm_Vertical, symbol Connector_Generic:Conn_02x08_Counter_Clockwise
- added J8: Conn_02x06_Counter_Clockwise, Connector_PinSocket_2.54mm:PinSocket_2x06_P2.54mm_Vertical, symbol Connector_Generic:Conn_02x06_Counter_Clockwise
Connections:
- net +3V3: now also J8.2 (Pin_2)
- net BT_GPIO6: now also J8.3 (Pin_3)
- net BT_PCM_CLK: now also J8.6 (Pin_6)
- net BT_PCM_IN: now also J8.7 (Pin_7)
- net BT_PCM_OUT: now also J8.9 (Pin_9)
- net BT_PCM_SYNC: now also J8.11 (Pin_11)
- net BT_SPI_MISO: now also J8.12 (Pin_12)
- net BT_SPI_MOSI: now also J8.8 (Pin_8)
- net BT_SPI_SCK: now also J8.10 (Pin_10)
- net BT_SPI_SS: now also J8.4 (Pin_4)
- net GND: now also J8.1 (Pin_1), J8.5 (Pin_5)
- net BT_MIC_BIAS: no longer names the net of J5.9 (Pin_9)
- net BT_MIC_L+: no longer names the net of J5.8 (Pin_8)
- net BT_MIC_L-: no longer names the net of J5.6 (Pin_6)
- net BT_MIC_R+: no longer names the net of J5.7 (Pin_7)
- net BT_MIC_R-: no longer names the net of J5.5 (Pin_5)
- no-connect marks 10 -> 15

Commit message: [HDW_51] FIX push button connector
Push button connector for power supply was not a holding
one and had to be changed to a holding one
PCB updated
Add of GND to some of the headers
Changed lines of the file:
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@@
   )
   (no_connect (at 137.16 78.105))
-  (no_connect (at 180.975 78.105))
+  (no_connect (at 180.975 73.025))
   (no_connect (at 153.035 142.24))
   (no_connect (at 59.69 158.115))
-  (no_connect (at 180.975 75.565))
+  (no_connect (at 180.975 70.485))
   (no_connect (at 59.69 163.195))
   (no_connect (at 180.975 83.185))
@@
     )
   )
-  (global_label "sys_onoff_i" (shape input) (at 180.975 70.485 0) (fields_autoplaced)
+  (global_label "sys_onoff_i" (shape input) (at 180.975 75.565 0) (fields_autoplaced)
     (effects (font (size 1.27 1.27)) (justify left))
-    (property "Intersheet References" "${INTERSHEET_REFS}" (id 0) (at 193.8505 70.4056 0)
+    (property "Intersheet References" "${INTERSHEET_REFS}" (id 0) (at 193.8505 75.4856 0)
       (effects (font (size 1.27 1.27)) (justify left) hide)
     )
@@
     )
   )
-  (global_label "sys_onoff_o" (shape input) (at 180.975 73.025 0) (fields_autoplaced)
+  (global_label "sys_onoff_o" (shape input) (at 180.975 78.105 0) (fields_autoplaced)
     (effects (font (size 1.27 1.27)) (justify left))
-    (property "Intersheet References" "${INTERSHEET_REFS}" (id 0) (at 194.3948 72.9456 0)
+    (property "Intersheet References" "${INTERSHEET_REFS}" (id 0) (at 194.3948 78.0256 0)
       (effects (font (size 1.27 1.27)) (justify left) hide)
     )
@@
       (reference "#PWR0166") (unit 1) (value "+3V3") (footprint "")
     )
+    (path "/f502a33a-d5e4-4b91-95a6-ac6a3abcb73b/4cee3fe2-7a49-4ea3-8dc4-0f7703510c06"
+      (reference "#PWR?") (unit 1) (value "GND") (footprint "")
+    )
+    (path "/f502a33a-d5e4-4b91-95a6-ac6a3abcb73b/557cc4f9-b02c-474b-91ea-cad4e36f9b5a"
+      (reference "#PWR?") (unit 1) (value "GND") (footprint "")
+    )
+    (path "/f502a33a-d5e4-4b91-95a6-ac6a3abcb73b/f4336b9f-7927-4d47-9509-dd3fd3c54804"
+      (reference "#PWR?") (unit 1) (value "GND") (footprint "")
+    )
     (path "/5a833556-9b2d-4a89-ade5-f769671d3e3c"
