File: 03_Development/Hardware/Proto_Bluetooth/Board_Bluetooth_radio_platform.kicad_sch (KiCad schematic)
At the start: 48 parts, among them J1 Conn_01x02, J10 Conn_01x03, J11 HMI_rotaryEncoder_1, J12 HMI_rotaryEncoder_1, J13 Conn_01x08_epaper, J19 Conn_01x02_rn52_usb, J2 Conn_01x08, J3 BT_RN52_connector_left, J4 Conn_01x02, J5 BT_RN52_connector_right, J6 FM_interface, J7 BT_debug_connector, J8 Conn_02x06_Counter_Clockwise, J9 SYS_debug_connector, SW1 SW_Push, U1 LM317_TO-220

Commit message: [HDW_55] FIX grounding of PCB for better gnd pane
Parts:
- added REF1, REF2, REF3, REF6: MountingHole, MountingHole:MountingHole_3.2mm_M3_DIN965, symbol Mechanical:MountingHole
- added REF4, REF5: MountingHole, MountingHole:MountingHole_2.5mm, symbol Mechanical:MountingHole
Changed lines of the file:
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@@
     (pin "9")
+  )
+  (symbol (lib_id "Mechanical:MountingHole") (at 137.795 52.07 0) (unit 1)
+    (in_bom yes) (on_board yes) (fields_autoplaced)
+    (property "Reference" "REF6" (id 0) (at 140.97 50.7999 0)
+      (effects (font (size 1.27 1.27)) (justify left))
+    )
+    (property "Value" "MountingHole" (id 1) (at 140.97 53.3399 0)
+      (effects (font (size 1.27 1.27)) (justify left) hide)
+    )
+    (property "Footprint" "MountingHole:MountingHole_3.2mm_M3_DIN965" (id 2) (at 137.795 52.07 0)
+      (effects (font (size 1.27 1.27)) hide)
+    )
+    (property "Datasheet" "~" (id 3) (at 137.795 52.07 0)
+      (effects (font (size 1.27 1.27)) hide)
+    )
   )
   (symbol (lib_id "power:GND") (at 261.62 60.325 0) (unit 1)
@@
     (pin "1")
   )
+  (symbol (lib_id "Mechanical:MountingHole") (at 137.795 40.64 0) (unit 1)
+    (in_bom yes) (on_board yes) (fields_autoplaced)
+    (property "Reference" "REF2" (id 0) (at 140.97 39.3699 0)
+      (effects (font (size 1.27 1.27)) (justify left))
+    )
+    (property "Value" "MountingHole" (id 1) (at 140.97 41.9099 0)
+      (effects (font (size 1.27 1.27)) (justify left))
+    )
+    (property "Footprint" "MountingHole:MountingHole_3.2mm_M3_DIN965" (id 2) (at 137.795 40.64 0)
+      (effects (font (size 1.27 1.27)) hide)
+    )
+    (property "Datasheet" "~" (id 3) (at 137.795 40.64 0)
+      (effects (font (size 1.27 1.27)) hide)
+    )
+  )
   (symbol (lib_id "Device:R") (at 252.73 70.485 90) (unit 1)
     (in_bom yes) (on_board yes)
@@
     )
     (pin "1")
+  )
+  (symbol (lib_id "Mechanical:MountingHole") (at 137.795 34.925 0) (unit 1)
+    (in_bom yes) (on_board yes) (fields_autoplaced)
+    (property "Reference" "REF1" (id 0) (at 140.97 33.6549 0)
+      (effects (font (size 1.27 1.27)) (justify left))
+    )
+    (property "Value" "MountingHole" (id 1) (at 140.97 36.1949 0)
+      (effects (font (size 1.27 1.27)) (justify left))
+    )
+    (property "Footprint" "MountingHole:MountingHole_3.2mm_M3_DIN965" (id 2) (at 137.795 34.925 0)
+      (effects (font (size 1.27 1.27)) hide)
+    )
+    (property "Datasheet" "~" (id 3) (at 137.795 34.925 0)
+      (effects (font (size 1.27 1.27)) hide)
+    )
   )
   (symbol (lib_id "Device:C_Polarized_US") (at 50.8 35.56 0) (unit 1)
@@
     (pin "1")
   )
+  (symbol (lib_id "Mechanical:MountingHole") (at 137.795 29.21 0) (unit 1)
+    (in_bom yes) (on_board yes) (fields_autoplaced)
+    (property "Reference" "REF5" (id 0) (at 140.97 27.9399 0)
+      (effects (font (size 1.27 1.27)) (justify left))
+    )
+    (property "Value" "MountingHole" (id 1) (at 140.97 30.4799 0)
+      (effects (font (size 1.27 1.27)) (justify left) hide)
+    )
+    (property "Footprint" "MountingHole:MountingHole_2.5mm" (id 2) (at 137.795 29.21 0)
+      (effects (font (size 1.27 1.27)) hide)
+    )
+    (property "Datasheet" "~" (id 3) (at 137.795 29.21 0)
+      (effects (font (size 1.27 1.27)) hide)
+    )
+  )
   (symbol (lib_id "Device:R") (at 28.575 127 0) (unit 1)
     (in_bom yes) (on_board yes)
@@
     (pin "3")
   )
+  (symbol (lib_id "Mechanical:MountingHole") (at 137.795 46.355 0) (unit 1)
+    (in_bom yes) (on_board yes) (fields_autoplaced)
+    (property "Reference" "REF3" (id 0) (at 140.97 45.0849 0)
+      (effects (font (size 1.27 1.27)) (justify left))
+    )
+    (property "Value" "MountingHole" (id 1) (at 140.97 47.6249 0)
+      (effects (font (size 1.27 1.27)) (justify left) hide)
+    )
+    (property "Footprint" "MountingHole:MountingHole_3.2mm_M3_DIN965" (id 2) (at 137.795 46.355 0)
+      (effects (font (size 1.27 1.27)) hide)
+    )
+    (property "Datasheet" "~" (id 3) (at 137.795 46.355 0)
+      (effects (font (size 1.27 1.27)) hide)
+    )
+  )
   (symbol (lib_id "Device:C") (at 238.76 81.28 0) (unit 1)
     (in_bom yes) (on_board yes)
@@
     )
     (pin "1")
+  )
+  (symbol (lib_id "Mechanical:MountingHole") (at 137.795 23.495 0) (unit 1)
+    (in_bom yes) (on_board yes) (fields_autoplaced)
+    (property "Reference" "REF4" (id 0) (at 140.97 22.2249 0)
+      (effects (font (size 1.27 1.27)) (justify left))
+    )
+    (property "Value" "MountingHole" (id 1) (at 140.97 24.7649 0)
+      (effects (font (size 1.27 1.27)) (justify left) hide)
+    )
+    (property "Footprint" "MountingHole:MountingHole_2.5mm" (id 2) (at 137.795 23.495 0)
+      (effects (font (size 1.27 1.27)) hide)
+    )
+    (property "Datasheet" "~" (id 3) (at 137.795 23.495 0)
+      (effects (font (size 1.27 1.27)) hide)
+    )
   )
   (symbol (lib_id "power:GND") (at 251.46 86.995 0) (unit 1)
@@
       (reference "#PWR0144") (unit 1) (value "GND") (footprint "")
     )
+    (path "/f502a33a-d5e4-4b91-95a6-ac6a3abcb73b/7953a399-cc2d-4ce4-9946-e52d90c54aac"
+      (reference "#PWR0145") (unit 1) (value "GND") (footprint "")
+    )
     (path "/f502a33a-d5e4-4b91-95a6-ac6a3abcb73b/5d5c2f63-1bc9-4a7f-a135-1bb26a50df72"
       (reference "#PWR0146") (unit 1) (value "GND") (footprint "")
@@
       (reference "#PWR0148") (unit 1) (value "GND") (footprint "")
     )
+    (path "/f502a33a-d5e4-4b91-95a6-ac6a3abcb73b/6a3fffbe-e83d-4276-a3c8-5994e1b8387c"
+      (reference "#PWR0149") (unit 1) (value "GND") (footprint "")
+    )
     (path "/f502a33a-d5e4-4b91-95a6-ac6a3abcb73b/16068be6-fd77-4fd5-b2cd-283ee84b3bec"
       (reference "#PWR0150") (unit 1) (value "GND") (footprint "")
@@
       (reference "#PWR0153") (unit 1) (value "GND") (footprint "")
     )
+    (path "/f502a33a-d5e4-4b91-95a6-ac6a3abcb73b/876b2b68-805f-4e62-a14b-0626ce4051fe"
+      (reference "#PWR0154") (unit 1) (value "GND") (footprint "")
+    )
     (path "/93984d3e-1049-40c4-85f7-3f9031f77d6e/3ecc4ac6-c427-462f-9dd1-91d4af84968d"
       (reference "#PWR0158") (unit 1) (value "+3V3") (footprint "")
@@
       (reference "R43") (unit 1) (value "10k") (footprint "Resistor_SMD:R_0805_2012Metric_Pad1.20x1.40mm_HandSolder")
     )
+    (path "/5775b7d3-efb6-41cd-a49a-c22ec5aad8c0"
+      (reference "REF1") (unit 1) (value "MountingHole") (footprint "MountingHole:MountingHole_3.2mm_M3_DIN965")
+    )
+    (path "/43d2825b-9d2e-4e56-a993-ded348020519"
+      (reference "REF2") (unit 1) (value "MountingHole") (footprint "MountingHole:MountingHole_3.2mm_M3_DIN965")
+    )
+    (path "/d2b544a7-d8e8-47e8-9a86-d54ee2b8f07b"
+      (reference "REF3") (unit 1) (value "MountingHole") (footprint "MountingHole:MountingHole_3.2mm_M3_DIN965")
+    )
+    (path "/e513f91e-cc26-43f9-93b9-f9058ea1464a"
+      (reference "REF4") (unit 1) (value "MountingHole") (footprint "MountingHole:MountingHole_2.5mm")
+    )
+    (path "/c45c05f7-025a-43be-aa8e-12e89e62a5cf"
+      (reference "REF5") (unit 1) (value "MountingHole") (footprint "MountingHole:MountingHole_2.5mm")
+    )
+    (path "/182165fa-3fdc-49ff-8161-498f546837d9"
+      (reference "REF6") (unit 1) (value "MountingHole") (footprint "MountingHole:MountingHole_3.2mm_M3_DIN965")
+    )
     (path "/521a4a83-0f29-4d03-acd6-c6cd2eb7ef82"
