File: 03_Development/Hardware/Proto_Bluetooth/Board_Bluetooth_radio_platform.kicad_sch (KiCad schematic)
At the start: 54 parts, among them J1 Conn_01x02, J10 Conn_01x03, J11 HMI_rotaryEncoder_1, J12 HMI_rotaryEncoder_1, J13 Conn_01x08_epaper, J19 Conn_01x02_rn52_usb, J2 Conn_01x08, J3 BT_RN52_connector_left, J4 Conn_01x02, J5 BT_RN52_connector_right, J6 FM_interface, J7 BT_debug_connector, J8 Conn_02x06_Counter_Clockwise, J9 SYS_debug_connector, SW1 SW_Push, U1 LM317_TO-220

Commit message: PROD Mark II - files sent to production
Modify mechanical placement of buttons and layout
Reduction of pull up/down resistances
Fix communication routing between modules and RP2040
Fix board size
Version: V1.1
Changed lines of the file:
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@@
   (junction (at 245.11 70.485) (diameter 0) (color 0 0 0 0)
-  )
-  (junction (at 238.76 86.36) (diameter 0) (color 0 0 0 0)
   )
   (junction (at 59.69 38.735) (diameter 0) (color 0 0 0 0)
@@
     (stroke (width 0) (type default) (color 0 0 0 0))
   )
-  (wire (pts (xy 238.76 86.36) (xy 238.76 86.995))
-    (stroke (width 0) (type default) (color 0 0 0 0))
-  )
   (wire (pts (xy 25.4 155.575) (xy 41.91 155.575))
     (stroke (width 0) (type default) (color 0 0 0 0))
@@
     (stroke (width 0) (type default) (color 0 0 0 0))
   )
-  (wire (pts (xy 238.76 85.09) (xy 238.76 86.36))
+  (wire (pts (xy 238.76 85.09) (xy 238.76 86.995))
     (stroke (width 0) (type default) (color 0 0 0 0))
   )
@@
     (pin "2")
   )
-  (symbol (lib_id "power:GND") (at 238.76 86.36 0) (unit 1)
+  (symbol (lib_id "power:GND") (at 238.76 86.995 0) (unit 1)
     (in_bom yes) (on_board yes) (fields_autoplaced)
-    (property "Reference" "#PWR0131" (id 0) (at 238.76 92.71 0)
-      (effects (font (size 1.27 1.27)) hide)
-    )
-    (property "Value" "GND" (id 1) (at 238.76 90.805 0))
-    (property "Footprint" "" (id 2) (at 238.76 86.36 0)
-      (effects (font (size 1.27 1.27)) hide)
-    )
-    (property "Datasheet" "" (id 3) (at 238.76 86.36 0)
-      (effects (font (size 1.27 1.27)) hide)
-    )
+    (property "Reference" "#PWR0131" (id 0) (at 238.76 93.345 0)
+      (effects (font (size 1.27 1.27)) hide)
+    )
+    (property "Value" "GND" (id 1) (at 238.76 91.44 0))
+    (property "Footprint" "" (id 2) (at 238.76 86.995 0)
+      (effects (font (size 1.27 1.27)) hide)
+    )
+    (property "Datasheet" "" (id 3) (at 238.76 86.995 0)
+      (effects (font (size 1.27 1.27)) hide)
+    )
