File: 03_Development/Hardware/Proto_Bluetooth/BtRadio_audioAmplifier.kicad_sch (KiCad schematic)
At the start: 26 parts, among them J14 Conn_01x03_fmModule_audioOutp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, J15 Conn_01x02_classD_SD, J20 Conn_01x05_toClassD, U3 TPA6112A2DGQ, U4 TS5A2234

Commit message: [HDW_39] Fix pull ups and pull down resistances
RP2040 internal's pull up/down are actually 80 kOhms
which is quite few. ALl filters and external pull up-down
are too high for them and incoming signal on RP2040
is too small.
Set all to either 4.7 kOhms or 10 kOhms
Parts:
- R28: value 100k -> 10k
Changed lines of the file:
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@@
     (in_bom yes) (on_board yes)
     (property "Reference" "R28" (id 0) (at 104.775 111.125 90))
-    (property "Value" "100k" (id 1) (at 102.235 109.855 90))
+    (property "Value" "10k" (id 1) (at 102.235 109.855 90))
     (property "Footprint" "Resistor_SMD:R_0805_2012Metric_Pad1.20x1.40mm_HandSolder" (id 2) (at 100.457 109.855 90)
       (effects (font (size 1.27 1.27)) hide)

Commit message: [HDW_54] FIX Bill Of Matierial for V1.1
FIX footprint of C15 and C16 from 0805 to 1210
Order all necessary parts from BOM
Parts:
- C16, C17: footprint Resistor_SMD:R_0805_2012Metric_Pad1.20x1.40mm_HandSolder -> Resistor_SMD:R_1206_3216Metric_Pad1.30x1.75mm_HandSolder
Changed lines of the file:
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@@
   (title_block
     (title "Audio amplifier")
-    (date "2023-01-13")
-    (rev "0.1")
+    (date "2023-09-27")
+    (rev "1.1")
     (company "DjenaDev")
   )
@@
     (property "Reference" "C17" (id 0) (at 92.075 93.98 90))
     (property "Value" "68u" (id 1) (at 99.695 93.98 90))
-    (property "Footprint" "Resistor_SMD:R_0805_2012Metric_Pad1.20x1.40mm_HandSolder" (id 2) (at 99.695 95.5548 0)
+    (property "Footprint" "Resistor_SMD:R_1206_3216Metric_Pad1.30x1.75mm_HandSolder" (id 2) (at 99.695 95.5548 0)
       (effects (font (size 1.27 1.27)) hide)
     )
@@
     (property "Reference" "C16" (id 0) (at 92.075 81.28 90))
     (property "Value" "68u" (id 1) (at 99.695 81.28 90))
-    (property "Footprint" "Resistor_SMD:R_0805_2012Metric_Pad1.20x1.40mm_HandSolder" (id 2) (at 99.695 82.8548 0)
-      (effects (font (size 1.27 1.27)) hide)
-    )
+    (property "Footprint" "Resistor_SMD:R_1206_3216Metric_Pad1.30x1.75mm_HandSolder" (id 2) (at 99.695 82.8548 0)
+      (effects (font (size 1.27 1.27)) hide)
+    )
